File: CPU.kicad_sch (KiCad schematic)
At the start: 207 parts, among them P1 Conn_02x36_Top_Bottom, P10 Conn_02x08_Counter_Clockwise, P2 Conn_02x13_Top_Bottom, P3 Conn_02x13_Top_Bottom, P4 Conn_02x08_Counter_Clockwise, P5 Conn_02x25_Counter_Clockwise, P6 Conn_02x25_Counter_Clockwise, P7 Conn_02x07_Counter_Clockwise, P8 Conn_02x08_Counter_Clockwise

Commit message: CPU: Part replacement
Some parts are not available, replaced with analogs
Parts:
- removed U_B13: 74LS471, Package_DIP:DIP-20_W7.62mm, symbol 74xx:74LS471
- removed U_L9: AM2911, Package_DIP:DIP-20_W7.62mm_Socket, symbol CPU:AM2911
- added U_B13.H, U_B13.L: 93427С, Package_DIP:DIP-20_W7.62mm, symbol 74xx:74LS471
- added U_L9: AM2909, Package_DIP:DIP-28_W15.24mm_Socket, symbol CPU:AM2909
Connections:
- net +5V: now also U_B13.H.16 (Vcc), U_B13.L.16 (Vcc), U_L9.1 (~{RE}), U_L9.28 (Vcc)
- net DataF.D_{0}: now also U_B13.L.12 (Q0)
- net DataF.D_{1}: now also U_B13.L.11 (Q1)
- net DataF.D_{2}: now also U_B13.L.10 (Q2)
- net DataF.D_{3}: now also U_B13.L.9 (Q3)
- net DataF.D_{4}: now also U_B13.H.12 (Q0)
- net DataF.D_{5}: now also U_B13.H.11 (Q1)
- net DataF.D_{6}: now also U_B13.H.10 (Q2)
- net DataF.D_{7}: now also U_B13.H.9 (Q3)
- net DataP.D_{0}: now also U_B13.H.5 (A0), U_B13.L.5 (A0)
- net DataP.D_{1}: now also U_B13.H.6 (A1), U_B13.L.6 (A1)
- net DataP.D_{2}: now also U_B13.H.7 (A2), U_B13.L.7 (A2)
- net DataP.D_{3}: now also U_B13.H.4 (A3), U_B13.L.4 (A3)
- net DataP.D_{4}: now also U_B13.H.3 (A4), U_B13.L.3 (A4)
- net DataP.D_{5}: now also U_B13.H.2 (A5), U_B13.L.2 (A5)
- net DataP.D_{6}: now also U_B13.H.1 (A6), U_B13.L.1 (A6)
- net DataP.D_{7}: now also U_B13.H.15 (A7), U_B13.L.15 (A7)
- net GND: now also U_B13.H.8 (GND), U_B13.L.8 (GND), U_L9.10 (OR_{1}), U_L9.12 (OR_{0}), U_L9.14 (GND), U_L9.2 (R_{3}), U_L9.3 (R_{2}), U_L9.4 (R_{1}), U_L9.5 (R_{0}), U_L9.6 (OR_{3}), U_L9.7 (D_{3}), U_L9.8 (OR_{2})
- net MW.D3_{0}: now also U_L9.13 (D_{0})
- net MW.D3_{1}: now also U_L9.11 (D_{1})
- net MW.D3_{2}: now also U_L9.9 (D_{2})
- net MW.D3_{4}: now also U_L9.26 (PUSH/~{POP})
- net MWS.A_{10}: now also U_L9.20 (Y_{2})
- net MWS.A_{8}: now also U_L9.18 (Y_{0})
- net MWS.A_{9}: now also U_L9.19 (Y_{1})
- net PROM_Disable: now also U_B13.H.14 (~{CE2}), U_B13.L.14 (~{CE2})
- net SEQ.S2_{1}: now also U_L9.17 (S_{1})
- net SEQ.SH_{0}: now also U_L9.16 (S_{0})
- net SEQ.~{FE}: now also U_L9.25 (~{FE})
- net SEQ.~{OE}: now also U_L9.22 (~{OE})
- net ~{ClockB_{0}}: now also U_L9.27 (CP)
- net ~{MAPROM_SEL}: now also U_B13.H.13 (~{CE1}), U_B13.L.13 (~{CE1})
- net ~{Reset_{1}}: now also U_L9.15 (~{ZERO})
- net at U_J7.24 (C_{n+4}): now also U_L9.23 (C_{n})

Commit message: CPU: Replace 8835
This part isn't available at all; so let's replace it with ls240 + ls244. ls240
looks the most electrically compatible in terms of current loads.
Parts:
- removed R13: 4.7k, Resistor_THT:R_Axial_DIN0207_L6.3mm_D2.5mm_P10.16mm_Horizontal, symbol Device:R
- removed U_A10, U_A4, U_A5, U_A6, U_A8, U_A9: 8835, Package_DIP:DIP-16_W7.62mm, symbol Interface:8835
- added R?: 4.7k, Resistor_THT:R_Axial_DIN0207_L6.3mm_D2.5mm_P10.16mm_Horizontal, symbol Device:R
- added UA9, U_A4, U_A6: 74LS244, symbol 74xx:74LS244
- added U_A10: 74LS240, Package_DIP:DIP-20_W7.62mm, symbol 74xx:74LS240
- added U_A5, U_A8: 74LS240, symbol 74xx:74LS240
Connections:
- net +5V: now also R?.1, UA9.20 (VCC), U_A10.20 (VCC), U_A4.20 (VCC), U_A5.20 (VCC), U_A6.20 (VCC), U_A8.20 (VCC)
- net Address.A_{0}: now also U_A4.11 (I0b), U_A5.11 (I0b)
- net Address.A_{10}: now also U_A6.15 (I2b), U_A8.15 (I2b)
- net Address.A_{11}: now also U_A6.17 (I3b), U_A8.17 (I3b)
- net Address.A_{1}: now also U_A4.13 (I1b), U_A5.13 (I1b)
- net Address.A_{2}: now also U_A4.15 (I2b), U_A5.15 (I2b)
- net Address.A_{3}: now also U_A4.17 (I3b), U_A5.17 (I3b)
- net Address.A_{4}: now also U_A4.2 (I0a), U_A5.2 (I0a)
- net Address.A_{5}: now also U_A4.4 (I1a), U_A5.4 (I1a)
- net Address.A_{6}: now also U_A4.6 (I2a), U_A5.6 (I2a)
- net Address.A_{7}: now also U_A4.8 (I3a), U_A5.8 (I3a)
- net Address.A_{8}: now also U_A6.11 (I0b), U_A8.11 (I0b)
- net Address.A_{9}: now also U_A6.13 (I1b), U_A8.13 (I1b)
- net CPL_{0}: now also U_A6.8 (I3a), U_A8.8 (I3a)
- net CPL_{1}: now also U_A6.6 (I2a), U_A8.6 (I2a)
- net CPL_{2}: now also U_A6.4 (I1a), U_A8.4 (I1a)
- net CPL_{3}: now also U_A6.2 (I0a), U_A8.2 (I0a)
- net DataP.D_{0}: now also UA9.9 (O0b), U_A4.9 (O0b), U_A6.9 (O0b)
- net DataP.D_{1}: now also UA9.7 (O1b), U_A4.7 (O1b), U_A6.7 (O1b)
- net DataP.D_{2}: now also UA9.5 (O2b), U_A4.5 (O2b), U_A6.5 (O2b)
- net DataP.D_{3}: now also UA9.3 (O3b), U_A4.3 (O3b), U_A6.3 (O3b)
- net DataP.D_{4}: now also UA9.18 (O0a), U_A4.18 (O0a), U_A6.12 (O3a)
- net DataP.D_{5}: now also UA9.16 (O1a), U_A4.16 (O1a), U_A6.14 (O2a)
- net DataP.D_{6}: now also UA9.12 (O3a), U_A4.14 (O2a), U_A6.16 (O1a)
- net DataP.D_{7}: now also UA9.14 (O2a), U_A4.12 (O3a), U_A6.18 (O0a)
- net GND: now also UA9.10 (GND), U_A10.10 (GND), U_A4.10 (GND), U_A5.1 (OEa), U_A5.10 (GND), U_A5.19 (OEb), U_A6.10 (GND), U_A8.10 (GND)
- net PTR.Q_{0}: now also UA9.11 (I0b), U_A10.11 (I0b)
- net PTR.Q_{1}: now also UA9.13 (I1b), U_A10.13 (I1b)
- net PTR.Q_{2}: now also UA9.15 (I2b), U_A10.15 (I2b)
- net PTR.Q_{3}: now also UA9.17 (I3b), U_A10.17 (I3b)
- net PTR.Q_{4}: now also UA9.2 (I0a), U_A10.2 (I0a)
- net PTR.Q_{5}: now also UA9.4 (I1a), U_A10.4 (I1a)
- net PTR.Q_{6}: now also UA9.8 (I3a), U_A10.8 (I3a)
- net Sys.~{A_{0}}: now also U_A5.9 (O0b)
- net Sys.~{A_{10}}: now also U_A8.5 (O2b)
- net Sys.~{A_{1}}: now also U_A5.7 (O1b)
- net Sys.~{A_{2}}: now also U_A5.5 (O2b)
- net Sys.~{A_{3}}: now also U_A5.3 (O3b)
- net Sys.~{A_{4}}: now also U_A5.18 (O0a)
- net Sys.~{A_{5}}: now also U_A5.16 (O1a)
- net Sys.~{A_{6}}: now also U_A5.14 (O2a)
- net Sys.~{A_{7}}: now also U_A5.12 (O3a)
- net Sys.~{A_{8}}: now also U_A8.9 (O0b)
- net Sys.~{A_{9}}: now also U_A8.7 (O1b)
- net Sys.~{CA_{15}}: now also U_A10.14 (O2a)
- net Sys.~{CPL_{0}}: now also U_A8.12 (O3a)
- net Sys.~{CPL_{1}}: now also U_A8.14 (O2a)
- net Sys.~{CPL_{2}}: now also U_A8.16 (O1a)
- net Sys.~{CPL_{3}}: now also U_A8.18 (O0a)
- net Sys.~{PA_{11}}: now also U_A10.9 (O0b)
- net Sys.~{PA_{12}}: now also U_A10.7 (O1b)
- net Sys.~{PA_{13}}: now also U_A10.5 (O2b)
- net Sys.~{PA_{14}}: now also U_A10.3 (O3b)
- net Sys.~{PA_{15}}: now also U_A10.18 (O0a)
- net Sys.~{PA_{16}}: now also U_A10.16 (O1a)
- net Sys.~{PA_{17}}: now also U_A10.12 (O3a)
- net ~{AddrHToData}: now also UA9.1 (OEa), UA9.19 (OEb)
- net ~{AddrHToSys}: now also U_A10.1 (OEa), U_A10.19 (OEb), U_A8.19 (OEb)
- net ~{AddrLToData}: now also U_A4.1 (OEa), U_A4.19 (OEb)
- net ~{AddrMToData}: now also U_A6.19 (OEb)
- net ~{H14_OE}: now also U_A6.1 (OEa)
- net CPL_Disable: now reaches U_E12.2
- net CPL_Disable: now also U_A8.1 (OEa)
- net at U_C8.12: now also UA9.6 (I2a), U_A10.6 (I2a)
- net ~{CPL_Disable}: no longer names the net of P4.14 (Pin_14), U_E12.1
- net ~{CPL_Disable}: now also R?.2
Other:
- moved on the sheet: U_A11, U_A12, U_A3C, U_A3D, U_A3E, U_C8A, U_C8B

Commit message: Get rid of 74ls378
This chip is rather rare and expensive here. Three can be replaced by 74ls379;
use 74ls377 instead of the remaining one (ALU flags register)

Analogs list populated and changed to a more proper encoding
Parts:
- removed U_D11, U_D9, U_J9, U_M12: 74LS378, Package_DIP:DIP-16_W7.62mm, symbol 74xx:74LS378
- added U_D11, U_M12: 74LS379, Package_DIP:DIP-16_W7.62mm, symbol 74xx:74LS379
- added U_D9: 74LS379, symbol 74xx:74LS379
- added U_J9: 74LS377, Package_SO:SOIC-20W_7.5x15.4mm_P1.27mm, symbol 74xx:74LS377
Connections:
- net +5V: now also U_D11.16 (VCC), U_D9.16 (VCC), U_J9.20 (VCC), U_M12.16 (VCC)
- net AFL.CARRY: now also U_J9.9 (Q3)
- net AFL.HALFC: now also U_J9.12 (Q4)
- net AFL.LZERO: now also U_J9.15 (Q5)
- net AFL.OVER: now also U_J9.6 (Q2)
- net AFL.SIGN: now also U_J9.5 (Q1)
- net AFL.ZERO: now also U_J9.14 (D5), U_J9.2 (Q0)
- net ALU.CARRY: now also U_J9.8 (D3)
- net ALU.HALFC: now also U_J9.13 (D4)
- net ALU.OVER: now also U_J9.7 (D2)
- net ALU.SIGN: now also U_J9.4 (D1)
- net ALU.ZERO: now also U_J9.3 (D0)
- net CCR.CARRY: now also U_M12.15 (Q3)
- net CCR.OVER: now also U_M12.10 (Q2)
- net CCR.SIGN: now also U_M12.7 (Q1)
- net CCR.ZERO: now also U_M12.2 (Q0)
- net CPL_{0}: now also U_D9.2 (Q0)
- net CPL_{1}: now also U_D9.7 (Q1)
- net CPL_{2}: now also U_D9.15 (Q3)
- net CPL_{3}: now also U_D9.10 (Q2)
- net DataF.D_{0}: now also U_D11.12 (D2)
- net DataF.D_{1}: now also U_D11.5 (D1)
- net DataF.D_{2}: now also U_D11.4 (D0)
- net DataF.D_{4}: now also U_D9.4 (D0)
- net DataF.D_{5}: now also U_D9.5 (D1)
- net DataF.D_{6}: now also U_D9.13 (D3)
- net DataF.D_{7}: now also U_D9.12 (D2)
- net GND: now also U_D11.13 (D3), U_D11.8 (GND), U_D9.8 (GND), U_J9.10 (GND), U_J9.17 (D6), U_J9.18 (D7), U_M12.8 (GND)
- net Page.B_{0}: now also U_D11.10 (Q2)
- net Page.B_{1}: now also U_D11.7 (Q1)
- net Page.B_{2}: now also U_D11.2 (Q0)
- net ~{ALU_Flags_EN}: now also U_J9.1 (~{E})
- net ~{CCR_EN}: now also U_M12.1 (~{E})
- net ~{ClockB_{1}}: now also U_J9.11 (CP), U_M12.9 (CP)
- net ~{ClockB_{2}}: now also U_D11.9 (CP), U_D9.9 (CP)
- net ~{Level_LD}: now also U_D9.1 (~{E})
- net ~{PTIndex_LD}: now also U_D11.1 (~{E})
- net at U_J11.5 (Z): now also U_M12.12 (D2)
- net at U_J10.5 (Z): now also U_M12.13 (D3)
- net at U_J12.9 (Zb): now also U_M12.4 (D0)
- net at U_J12.7 (Za): now also U_M12.5 (D1)
- no-connect marks 83 -> 91
