File: CPU.kicad_sch (KiCad schematic)
At the start: 208 parts, among them J1 Conn_02x36_Odd_Even, P10 Conn_02x08_Counter_Clockwise, P2 Conn_02x13_Top_Bottom, P3 Conn_02x13_Top_Bottom, P4 Conn_02x08_Counter_Clockwise, P5 Conn_02x25_Counter_Clockwise, P6 Conn_02x25_Counter_Clockwise, P7 Conn_02x07_Counter_Clockwise, P8 Conn_02x08_Counter_Clockwise

Commit message: Changed twist on uCode read buffers
This yields much more optimal PCB layout
Parts:
- renumbered U_BL13 to U_BH13
Connections:
- net MW.A6_{2}: now also U_K5.12 (Q4); no longer U_K5.6 (Q2)
- net MW.A6_{3}: now also U_K5.15 (Q5); no longer U_K5.9 (Q3)
- net MW.A6_{4}: now also U_K5.6 (Q2); no longer U_K5.12 (Q4)
- net MW.A6_{5}: now also U_K5.9 (Q3); no longer U_K5.15 (Q5)
- net MW.B5_{2}: now also U_F5.12 (Q4); no longer U_F5.6 (Q2)
- net MW.B5_{3}: now also U_F5.15 (Q5); no longer U_F5.9 (Q3)
- net MW.B5_{4}: now also U_F5.6 (Q2); no longer U_F5.12 (Q4)
- net MW.B5_{5}: now also U_F5.9 (Q3); no longer U_F5.15 (Q5)
- net MW.C4_{2}: now also U_H5.12 (Q4); no longer U_H5.6 (Q2)
- net MW.C4_{3}: now also U_H5.15 (Q5); no longer U_H5.9 (Q3)
- net MW.C4_{4}: now also U_H5.6 (Q2); no longer U_H5.12 (Q4)
- net MW.C4_{5}: now also U_H5.9 (Q3); no longer U_H5.15 (Q5)
- net MW.D3_{2}: now also U_L5.12 (Q4); no longer U_L5.6 (Q2)
- net MW.D3_{3}: now also U_L5.15 (Q5); no longer U_L5.9 (Q3)
- net MW.D3_{4}: now also U_L5.6 (Q2); no longer U_L5.12 (Q4)
- net MW.D3_{5}: now also U_L5.9 (Q3); no longer U_L5.15 (Q5)
- net MW.E2_{2}: now also U_M5.12 (Q4); no longer U_M5.6 (Q2)
- net MW.E2_{3}: now also U_M5.15 (Q5); no longer U_M5.9 (Q3)
- net MW.E2_{4}: now also U_M5.6 (Q2); no longer U_M5.12 (Q4)
- net MW.E2_{5}: now also U_M5.9 (Q3); no longer U_M5.15 (Q5)
- net MW.F1_{2}: now also U_J5.12 (Q4); no longer U_J5.6 (Q2)
- net MW.F1_{3}: now also U_J5.15 (Q5); no longer U_J5.9 (Q3)
- net MW.F1_{4}: now also U_J5.6 (Q2); no longer U_J5.12 (Q4)
- net MW.F1_{5}: now also U_J5.9 (Q3); no longer U_J5.15 (Q5)
- net MWR.A6_{2}: now also U_K5.13 (D4); no longer U_K5.7 (D2)
- net MWR.A6_{3}: now also U_K5.14 (D5); no longer U_K5.8 (D3)
- net MWR.A6_{4}: now also U_K5.7 (D2); no longer U_K5.13 (D4)
- net MWR.A6_{5}: now also U_K5.8 (D3); no longer U_K5.14 (D5)
- net MWR.B5_{2}: now also U_F5.13 (D4); no longer U_F5.7 (D2)
- net MWR.B5_{3}: now also U_F5.14 (D5); no longer U_F5.8 (D3)
- net MWR.B5_{4}: now also U_F5.7 (D2); no longer U_F5.13 (D4)
- net MWR.B5_{5}: now also U_F5.8 (D3); no longer U_F5.14 (D5)
- net MWR.C4_{2}: now also U_H5.13 (D4); no longer U_H5.7 (D2)
- net MWR.C4_{3}: now also U_H5.14 (D5); no longer U_H5.8 (D3)
- net MWR.C4_{4}: now also U_H5.7 (D2); no longer U_H5.13 (D4)
- net MWR.C4_{5}: now also U_H5.8 (D3); no longer U_H5.14 (D5)
- net MWR.D3_{2}: now also U_L5.13 (D4); no longer U_L5.7 (D2)
- net MWR.D3_{3}: now also U_L5.14 (D5); no longer U_L5.8 (D3)
- net MWR.D3_{4}: now also U_L5.7 (D2); no longer U_L5.13 (D4)
- net MWR.D3_{5}: now also U_L5.8 (D3); no longer U_L5.14 (D5)
- net MWR.E2_{2}: now also U_M5.13 (D4); no longer U_M5.7 (D2)
- net MWR.E2_{3}: now also U_M5.14 (D5); no longer U_M5.8 (D3)
- net MWR.E2_{4}: now also U_M5.7 (D2); no longer U_M5.13 (D4)
- net MWR.E2_{5}: now also U_M5.8 (D3); no longer U_M5.14 (D5)
- net MWR.F1_{2}: now also U_J5.13 (D4); no longer U_J5.7 (D2)
- net MWR.F1_{3}: now also U_J5.14 (D5); no longer U_J5.8 (D3)
- net MWR.F1_{4}: now also U_J5.7 (D2); no longer U_J5.13 (D4)
- net MWR.F1_{5}: now also U_J5.8 (D3); no longer U_J5.14 (D5)
Other:
- note added: "These line twists help to optimize the PCB layout"
