File: CPU.kicad_pcb (KiCad board)
At the start: 4 copper layers, 212 parts, among them J1 Conn_02x36_Odd_Even, P10 Conn_02x08_Counter_Clockwise, P2 Conn_02x13_Top_Bottom, P3 Conn_02x13_Top_Bottom, P4 Conn_02x08_Counter_Clockwise, P5 Conn_02x25_Counter_Clockwise, P6 Conn_02x25_Counter_Clockwise, P7 Conn_02x07_Counter_Clockwise, P8 Conn_02x08_Counter_Clockwise

Commit message: DIP layout prototype
Parts arranged
Parts:
- added REF**: BUS_EE200, Connector_PCBEdge:BUS_EE200, F.Cu at (379.0, 50.0)
- C39: footprint Capacitor_THT:CP_Radial_D8.0mm_P3.80mm -> Capacitor_THT:CP_Radial_D8.0mm_P2.50mm
- J1: footprint Connector_PinHeader_2.54mm:PinHeader_2x36_P2.54mm_Horizontal -> Connector_PinHeader_2.54mm:PinHeader_2x35_P2.54mm_Vertical
- U_A1, U_B15, U_E15, U_F12, U_L10, U_M9: footprint Package_SO:SOIC-16W_7.5x12.8mm_P1.27mm -> Package_DIP:DIP-14_W7.62mm
- U_A15, U_A3, U_C10, U_C7, U_C8, U_D10, U_E12, U_E14, U_E8, U_J6, U_K12: footprint Package_SO:SOIC-14_3.9x8.7mm_P1.27mm -> Package_DIP:DIP-14_W7.62mm
- U_A4, U_A6, U_A9, U_C13, U_C9, U_D13, U_F5, U_H5, U_J5, U_J9, U_K5, U_L5, U_M5: footprint Package_SO:SOIC-20W_7.5x15.4mm_P1.27mm -> Package_DIP:DIP-20_W7.62mm
- U_B11, U_B12, U_B7, U_B8, U_D12, U_E10, U_E11, U_F14, U_K10, U_K6, U_L14, U_L6: footprint Package_SO:SO-14_5.3x10.2mm_P1.27mm -> Package_DIP:DIP-14_W7.62mm
- U_B3, U_B4, U_C14, U_C3, U_C4, U_D6, U_H14, U_J10, U_J11, U_K9, U_L11: footprint Package_SO:SO-16_5.3x10.2mm_P1.27mm -> Package_DIP:DIP-16_W7.62mm
- U_BH13, U_BL13: value 93427С -> 93427C
- U_C11, U_C12: footprint Package_SO:SOIC-16W_7.5x10.3mm_P1.27mm -> Package_DIP:DIP-16_W7.62mm
- U_D2, U_D3, U_D4, U_D5, U_D7, U_E5, U_E6, U_E7, U_F11, U_F13, U_F6, U_H11, U_H12, U_H6, U_J12, U_J13, U_K11, U_K13, U_L13, U_M13: footprint Package_SO:SOIC-16W_7.5x12.8mm_P1.27mm -> Package_DIP:DIP-16_W7.62mm
- U_D8, U_H13: footprint Package_SO:SOIC-14W_7.5x9mm_P1.27mm -> Package_DIP:DIP-14_W7.62mm
- XTAL1: footprint Crystal:Crystal_HC52-U_Horizontal -> Crystal:Crystal_HC18-U_Vertical
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Connections:
- C1 pad 1: +5V -> (no net)
- C1 pad 2: GND -> (no net)
- C10 pad 1: +5V -> (no net)
- C10 pad 2: GND -> (no net)
- C11 pad 1: +5V -> (no net)
- C11 pad 2: GND -> (no net)
- C12 pad 1: +5V -> (no net)
- C12 pad 2: GND -> (no net)
- C13 pad 1: +5V -> (no net)
- C13 pad 2: GND -> (no net)
- C14 pad 1: +5V -> (no net)
- C14 pad 2: GND -> (no net)
- C15 pad 1: +5V -> (no net)
- C15 pad 2: GND -> (no net)
- C16 pad 1: +5V -> (no net)
- C16 pad 2: GND -> (no net)
- C17 pad 1: +5V -> (no net)
- C17 pad 2: GND -> (no net)
- C18 pad 1: +5V -> (no net)
- C18 pad 2: GND -> (no net)
- C19 pad 1: +5V -> (no net)
- C19 pad 2: GND -> (no net)
- C2 pad 1: +5V -> (no net)
- C2 pad 2: GND -> (no net)
- C20 pad 1: +5V -> (no net)
- C20 pad 2: GND -> (no net)
- C21 pad 1: +5V -> (no net)
- C21 pad 2: GND -> (no net)
- C22 pad 1: +5V -> (no net)
- C22 pad 2: GND -> (no net)
- C23 pad 1: +5V -> (no net)
- C23 pad 2: GND -> (no net)
- C24 pad 1: +5V -> (no net)
- C24 pad 2: GND -> (no net)
- C25 pad 1: +5V -> (no net)
- C25 pad 2: GND -> (no net)
- C26 pad 1: +5V -> (no net)
- C26 pad 2: GND -> (no net)
- C27 pad 1: +5V -> (no net)
- C27 pad 2: GND -> (no net)
- C28 pad 1: +5V -> (no net)
- C28 pad 2: GND -> (no net)
- C29 pad 1: +5V -> (no net)
- C29 pad 2: GND -> (no net)
- C3 pad 1: +5V -> (no net)
- C3 pad 2: GND -> (no net)
- C30 pad 1: +5V -> (no net)
- C30 pad 2: GND -> (no net)
- C31 pad 1: +5V -> (no net)
- C31 pad 2: GND -> (no net)
- C32 pad 1: +5V -> (no net)
- C32 pad 2: GND -> (no net)
- C33 pad 1: +5V -> (no net)
- C33 pad 2: GND -> (no net)
- C34 pad 1: +5V -> (no net)
- C34 pad 2: GND -> (no net)
- C35 pad 1: +5V -> (no net)
- C35 pad 2: GND -> (no net)
- C36 pad 1: +5V -> (no net)
- C36 pad 2: GND -> (no net)
- C37 pad 1: +5V -> (no net)
- C37 pad 2: GND -> (no net)
- C38 pad 1: +5V -> (no net)
- C38 pad 2: GND -> (no net)
- C39 pad 1: VERIFY_CR1 -> (no net)
- C39 pad 2: GND -> (no net)
- C4 pad 1: +5V -> (no net)
- C4 pad 2: GND -> (no net)
- C40 pad 1: +5V -> (no net)
- C40 pad 2: GND -> (no net)
- C41 pad 1: +5V -> (no net)
- C41 pad 2: GND -> (no net)
- C42 pad 1: +5V -> (no net)
- C42 pad 2: GND -> (no net)
- C43 pad 1: +5V -> (no net)
- C43 pad 2: GND -> (no net)
- C44 pad 1: +5V -> (no net)
- C44 pad 2: GND -> (no net)
- C45 pad 1: +5V -> (no net)
- C45 pad 2: GND -> (no net)
- C46 pad 1: +5V -> (no net)
- C46 pad 2: GND -> (no net)
- C47 pad 1: +5V -> (no net)
- C47 pad 2: GND -> (no net)
- C48 pad 1: +5V -> (no net)
- C48 pad 2: GND -> (no net)
- C49 pad 1: +5V -> (no net)
- C49 pad 2: GND -> (no net)
- C5 pad 1: +5V -> (no net)
- C5 pad 2: GND -> (no net)
- C50 pad 1: +5V -> (no net)
- C50 pad 2: GND -> (no net)
- C51 pad 1: +5V -> (no net)
- C51 pad 2: GND -> (no net)
- C52 pad 1: +5V -> (no net)
- C52 pad 2: GND -> (no net)
- C53 pad 1: +5V -> (no net)
- C53 pad 2: GND -> (no net)
- C54 pad 1: +5V -> (no net)
- C54 pad 2: GND -> (no net)
- C6 pad 1: +5V -> (no net)
- C6 pad 2: GND -> (no net)
- C7 pad 1: +5V -> (no net)
- C7 pad 2: GND -> (no net)
- C8 pad 1: +5V -> (no net)
- C8 pad 2: GND -> (no net)
- C9 pad 1: +5V -> (no net)
- C9 pad 2: GND -> (no net)
- CR1 pad 1: +5V -> (no net)
- CR1 pad 2: VERIFY_CR1 -> (no net)
- DSW1 pad 1: /Sys.Reset -> (no net)
- DSW1 pad 10: GND -> (no net)
- DSW1 pad 11: GND -> (no net)
- DSW1 pad 12: GND -> (no net)
- DSW1 pad 13: GND -> (no net)
- DSW1 pad 14: GND -> (no net)
- DSW1 pad 15: GND -> (no net)
- DSW1 pad 16: GND -> (no net)
- DSW1 pad 2: /SW_3 -> (no net)
- DSW1 pad 3: /SW_2 -> (no net)
- DSW1 pad 4: /SW_1 -> (no net)
- DSW1 pad 5: /SW_R -> (no net)
- DSW1 pad 6: /SW_H -> (no net)
- DSW1 pad 7: /SW_I -> (no net)
- DSW1 pad 8: /SW_O -> (no net)
- DSW1 pad 9: GND -> (no net)
- J1 pad 1: GND -> (no net)
- J1 pad 10: unconnected-(J1-Pad10) -> (no net)
- J1 pad 11: /Sys.~{A_{1}} -> (no net)
- J1 pad 12: /Sys.~{RDIN} -> (no net)
- J1 pad 13: /Sys.~{A_{2}} -> (no net)
- J1 pad 14: /Sys.~{WTIN} -> (no net)
- J1 pad 15: /Sys.~{A_{3}} -> (no net)
- J1 pad 16: /Sys.~{DRDY} -> (no net)
- J1 pad 17: /Sys.~{A_{4}} -> (no net)
- J1 pad 18: /Sys.~{RA_{14}} -> (no net)
- J1 pad 19: /Sys.~{A_{5}} -> (no net)
- J1 pad 2: GND -> (no net)
- J1 pad 20: /Sys.~{RA_{12}} -> (no net)
- J1 pad 21: /Sys.~{A_{6}} -> (no net)
- J1 pad 22: /Sys.~{APRE} -> (no net)
- J1 pad 23: /Sys.~{A_{7}} -> (no net)
- J1 pad 24: /Sys.~{RA_{13}} -> (no net)
- J1 pad 25: /Sys.~{A_{8}} -> (no net)
- J1 pad 26: /Sys.~{INR1} -> (no net)
- J1 pad 27: /Sys.~{A_{9}} -> (no net)
- J1 pad 28: /Sys.~{INR2} -> (no net)
- J1 pad 29: /Sys.~{A_{10}} -> (no net)
- J1 pad 3: +5V -> (no net)
- J1 pad 30: /Sys.~{INR3} -> (no net)
- J1 pad 31: /Sys.~{PA_{11}} -> (no net)
- J1 pad 32: /Sys.~{INR0} -> (no net)
- J1 pad 33: /Sys.~{PA_{12}} -> (no net)
- J1 pad 34: /Sys.~{RA_{15}} -> (no net)
- J1 pad 35: /Sys.~{PA_{13}} -> (no net)
- J1 pad 36: /Sys.~{CPL_{0}} -> (no net)
- J1 pad 37: /Sys.~{PA_{14}} -> (no net)
- J1 pad 38: /Sys.~{CPL_{1}} -> (no net)
- J1 pad 39: /Sys.~{CA_{15}} -> (no net)
- J1 pad 4: +5V -> (no net)
- J1 pad 40: /Sys.~{CPL_{2}} -> (no net)
- J1 pad 41: /Sys.~{D_{0}} -> (no net)
- J1 pad 42: /Sys.~{CPL_{3}} -> (no net)
- J1 pad 43: /Sys.~{D_{1}} -> (no net)
- J1 pad 44: /Sys.~{RA_{11}} -> (no net)
- J1 pad 45: /Sys.~{D_{2}} -> (no net)
- J1 pad 46: /Sys.~{PA_{15}} -> (no net)
- J1 pad 47: /Sys.~{D_{3}} -> (no net)
- J1 pad 48: /Sys.~{PA_{16}} -> (no net)
- J1 pad 49: /Sys.~{D_{4}} -> (no net)
- J1 pad 5: unconnected-(J1-Pad5) -> (no net)
- J1 pad 50: /Sys.~{PA_{17}} -> (no net)
- J1 pad 51: /Sys.~{D_{5}} -> (no net)
- J1 pad 52: /Sys.~{PTR7_oc} -> (no net)
- J1 pad 53: /Sys.~{D_{6}} -> (no net)
- J1 pad 54: /Sys.~{INTREQ} -> (no net)
- J1 pad 55: /Sys.~{D_{7}} -> (no net)
- J1 pad 56: /Sys.~{MemFault} -> (no net)
- J1 pad 57: /Sys.~{ParityTest} -> (no net)
- J1 pad 58: /Sys.~{INTACK} -> (no net)
- J1 pad 59: Net-(J1-Pad59) -> (no net)
- J1 pad 6: +12V -> (no net)
- J1 pad 60: Net-(J1-Pad59) -> (no net)
- J1 pad 61: /Sys.5MHz -> (no net)
- J1 pad 62: Net-(J1-Pad59) -> (no net)
- J1 pad 63: /Sys.Reset -> (no net)
- J1 pad 64: Net-(J1-Pad59) -> (no net)
- J1 pad 65: Net-(J1-Pad59) -> (no net)
- J1 pad 66: Net-(J1-Pad59) -> (no net)
- J1 pad 67: unconnected-(J1-Pad67) -> (no net)
- J1 pad 68: -12V -> (no net)
- J1 pad 69: +5V -> (no net)
- J1 pad 7: unconnected-(J1-Pad7) -> (no net)
- J1 pad 70: +5V -> (no net)
- J1 pad 8: unconnected-(J1-Pad8) -> (no net)
- J1 pad 9: /Sys.~{A_{0}} -> (no net)
- JP1 pad 1: Net-(JP1-Pad1) -> (no net)
- JP1 pad 2: /PTR.~{Q_{7}} -> (no net)
- JP1 pad 3: Net-(JP1-Pad3) -> (no net)
- P10 pad 1: /PTR.Q_{0} -> (no net)
- P10 pad 10: Address.A_{15} -> (no net)
- P10 pad 11: Address.A_{15} -> (no net)
- P10 pad 12: Address.A_{15} -> (no net)
- P10 pad 13: Address.A_{14} -> (no net)
- P10 pad 14: Address.A_{13} -> (no net)
- P10 pad 15: Address.A_{12} -> (no net)
- P10 pad 16: Address.A_{11} -> (no net)
- P10 pad 2: /PTR.Q_{1} -> (no net)
- P10 pad 3: /PTR.Q_{2} -> (no net)
- P10 pad 4: /PTR.Q_{3} -> (no net)
- P10 pad 5: /PTR.Q_{4} -> (no net)
- P10 pad 6: /PTR.Q_{5} -> (no net)
- P10 pad 7: /PTR.Q_{6} -> (no net)
- P10 pad 8: /PTR.Q_{7} -> (no net)
- P10 pad 9: unconnected-(P10-Pad9) -> (no net)
- P2 pad 1: unconnected-(P2-Pad1) -> (no net)
- P2 pad 10: GND -> (no net)
- P2 pad 11: /DMA.~{Enable} -> (no net)
- P2 pad 12: GND -> (no net)
- P2 pad 13: Net-(P2-Pad13) -> (no net)
- P2 pad 14: GND -> (no net)
- P2 pad 15: /DMA.~{BusReadReady} -> (no net)
- P2 pad 16: GND -> (no net)
- P2 pad 17: /DMA.~{BusWriteOE} -> (no net)
- P2 pad 18: GND -> (no net)
- P2 pad 19: /DMA.~{StartCycle} -> (no net)
- P2 pad 2: GND -> (no net)
- P2 pad 20: GND -> (no net)
- P2 pad 21: /DMA.Write -> (no net)
- P2 pad 22: GND -> (no net)
- P2 pad 23: /DMA.~{INTRequest} -> (no net)
- P2 pad 24: GND -> (no net)
- P2 pad 25: /DMA.~{Request} -> (no net)
- P2 pad 26: GND -> (no net)
- P2 pad 3: /DMA.~{AddressControl} -> (no net)
- P2 pad 4: GND -> (no net)
- P2 pad 5: Net-(P2-Pad5) -> (no net)
- P2 pad 6: GND -> (no net)
- P2 pad 7: Net-(P2-Pad7) -> (no net)
- P2 pad 8: GND -> (no net)
- P2 pad 9: /DMA.~{End} -> (no net)
- P3 pad 1: FP.~{HALT} -> (no net)
- P3 pad 10: GND -> (no net)
- P3 pad 11: Net-(P3-Pad11) -> (no net)
- P3 pad 12: GND -> (no net)
- P3 pad 13: Net-(P3-Pad13) -> (no net)
- P3 pad 14: GND -> (no net)
- P3 pad 15: /SW_2 -> (no net)
- P3 pad 16: +5V -> (no net)
- P3 pad 17: /~{ResetFlag} -> (no net)
- P3 pad 18: +5V -> (no net)
- P3 pad 19: Net-(P3-Pad19) -> (no net)
- P3 pad 2: unconnected-(P3-Pad2) -> (no net)
- P3 pad 20: +5V -> (no net)
- P3 pad 21: Net-(P3-Pad21) -> (no net)
- P3 pad 22: +5V -> (no net)
- P3 pad 23: Net-(P3-Pad23) -> (no net)
- P3 pad 24: +5V -> (no net)
- P3 pad 25: FP.RTI -> (no net)
- P3 pad 26: +5V -> (no net)
- P3 pad 3: FP.~{RUN} -> (no net)
- P3 pad 4: /R4_7 -> (no net)
- P3 pad 5: Net-(P3-Pad5) -> (no net)
- P3 pad 6: Net-(P3-Pad6) -> (no net)
- P3 pad 7: /SW_O -> (no net)
- P3 pad 8: GND -> (no net)
- P3 pad 9: Net-(P3-Pad9) -> (no net)
- P4 pad 1: GND -> (no net)
- P4 pad 10: DataF.D_{4} -> (no net)
- P4 pad 11: DataF.D_{5} -> (no net)
- P4 pad 12: DataF.D_{6} -> (no net)
- P4 pad 13: DataF.D_{7} -> (no net)
- P4 pad 14: Net-(P4-Pad14) -> (no net)
- P4 pad 15: GND -> (no net)
- P4 pad 16: GND -> (no net)
- P4 pad 2: GND -> (no net)
- P4 pad 3: DataF.D_{0} -> (no net)
- P4 pad 4: DataF.D_{1} -> (no net)
- P4 pad 5: DataF.D_{2} -> (no net)
- P4 pad 6: DataF.D_{3} -> (no net)
- P4 pad 7: /P4_7 -> (no net)
- P4 pad 8: +5V -> (no net)
- P4 pad 9: +5V -> (no net)
- P5 pad 1: /MWR.H0_{6} -> (no net)
- P5 pad 10: /MWR.H0_{1} -> (no net)
- P5 pad 11: GND -> (no net)
- P5 pad 12: /MWR.H0_{0} -> (no net)
- P5 pad 13: GND -> (no net)
- P5 pad 14: /MWR.B5_{7} -> (no net)
- P5 pad 15: GND -> (no net)
- P5 pad 16: /MWR.B5_{6} -> (no net)
- P5 pad 17: GND -> (no net)
- P5 pad 18: /MWR.B5_{5} -> (no net)
- P5 pad 19: GND -> (no net)
- P5 pad 2: /MWR.H0_{5} -> (no net)
- P5 pad 20: /MWR.B5_{4} -> (no net)
- P5 pad 21: GND -> (no net)
- P5 pad 22: /MWR.B5_{3} -> (no net)
- P5 pad 23: GND -> (no net)
- P5 pad 24: /MWR.B5_{2} -> (no net)
- P5 pad 25: GND -> (no net)
- P5 pad 26: /MWR.B5_{1} -> (no net)
- P5 pad 27: GND -> (no net)
- P5 pad 28: /MWR.B5_{0} -> (no net)
- P5 pad 29: GND -> (no net)
- P5 pad 3: /MWR.H0_{7} -> (no net)
- P5 pad 30: /MWR.C4_{7} -> (no net)
- P5 pad 31: GND -> (no net)
- P5 pad 32: /MWR.C4_{6} -> (no net)
- P5 pad 33: GND -> (no net)
- P5 pad 34: /MWR.C4_{5} -> (no net)
- P5 pad 35: GND -> (no net)
- P5 pad 36: /MWR.C4_{4} -> (no net)
- P5 pad 37: GND -> (no net)
- P5 pad 38: /MWR.C4_{3} -> (no net)
- P5 pad 39: GND -> (no net)
- P5 pad 4: /MWR.H0_{4} -> (no net)
- P5 pad 40: /MWR.C4_{2} -> (no net)
- P5 pad 41: GND -> (no net)
- P5 pad 42: /MWR.C4_{1} -> (no net)
- P5 pad 43: GND -> (no net)
- P5 pad 44: /MWR.C4_{0} -> (no net)
- P5 pad 45: GND -> (no net)
- P5 pad 46: /MWR.F1_{7} -> (no net)
- P5 pad 47: GND -> (no net)
- P5 pad 48: /MWR.F1_{6} -> (no net)
- P5 pad 49: /MWR.F1_{4} -> (no net)
- P5 pad 5: GND -> (no net)
- P5 pad 50: /MWR.F1_{5} -> (no net)
- P5 pad 6: /MWR.H0_{3} -> (no net)
- P5 pad 7: GND -> (no net)
- P5 pad 8: /MWR.H0_{2} -> (no net)
- P5 pad 9: GND -> (no net)
- P6 pad 1: /MWR.F1_{2} -> (no net)
- P6 pad 10: /MWR.A6_{5} -> (no net)
- P6 pad 11: GND -> (no net)
- P6 pad 12: /MWR.A6_{4} -> (no net)
- P6 pad 13: GND -> (no net)
- P6 pad 14: /MWR.A6_{3} -> (no net)
- P6 pad 15: GND -> (no net)
- P6 pad 16: /MWR.A6_{2} -> (no net)
- P6 pad 17: GND -> (no net)
- P6 pad 18: /MWR.A6_{1} -> (no net)
- P6 pad 19: GND -> (no net)
- P6 pad 2: /MWR.F1_{1} -> (no net)
- P6 pad 20: /MWR.A6_{0} -> (no net)
- P6 pad 21: GND -> (no net)
- P6 pad 22: /MWR.D3_{7} -> (no net)
- P6 pad 23: GND -> (no net)
- P6 pad 24: /MWR.D3_{6} -> (no net)
- P6 pad 25: GND -> (no net)
- P6 pad 26: /MWR.D3_{5} -> (no net)
- P6 pad 27: GND -> (no net)
- P6 pad 28: /MWR.D3_{4} -> (no net)
- P6 pad 29: GND -> (no net)
- P6 pad 3: /MWR.F1_{3} -> (no net)
- P6 pad 30: /MWR.D3_{3} -> (no net)
- P6 pad 31: GND -> (no net)
- P6 pad 32: /MWR.D3_{2} -> (no net)
- P6 pad 33: GND -> (no net)
- P6 pad 34: /MWR.D3_{1} -> (no net)
- P6 pad 35: GND -> (no net)
- P6 pad 36: /MWR.D3_{0} -> (no net)
- P6 pad 37: GND -> (no net)
- P6 pad 38: /MWR.E2_{7} -> (no net)
- P6 pad 39: GND -> (no net)
- P6 pad 4: /MWR.F1_{0} -> (no net)
- P6 pad 40: /MWR.E2_{6} -> (no net)
- P6 pad 41: GND -> (no net)
- P6 pad 42: /MWR.E2_{5} -> (no net)
- P6 pad 43: GND -> (no net)
- P6 pad 44: /MWR.E2_{4} -> (no net)
- P6 pad 45: GND -> (no net)
- P6 pad 46: /MWR.E2_{3} -> (no net)
- P6 pad 47: GND -> (no net)
- P6 pad 48: /MWR.E2_{2} -> (no net)
- P6 pad 49: /MWR.E2_{0} -> (no net)
- P6 pad 5: GND -> (no net)
- P6 pad 50: /MWR.E2_{1} -> (no net)
- P6 pad 6: /MWR.A6_{7} -> (no net)
- P6 pad 7: GND -> (no net)
- P6 pad 8: /MWR.A6_{6} -> (no net)
- P6 pad 9: GND -> (no net)
- P7 pad 1: P7_1 -> (no net)
- P7 pad 10: GND -> (no net)
- P7 pad 11: GND -> (no net)
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Other:
- board outline added: 364 x 203 mm

Commit message: Part of routed layout
A successful manually routed part: sequencer ROMs and buffers.
Parts:
- C39: footprint Capacitor_THT:CP_Radial_D8.0mm_P2.50mm -> Capacitor_THT:CP_Axial_L18.0mm_D8.0mm_P25.00mm_Horizontal
- J1: footprint Connector_PinHeader_2.54mm:PinHeader_2x35_P2.54mm_Vertical -> Connector_PinHeader_2.54mm:PinHeader_2x36_P2.54mm_Horizontal
- XTAL1: footprint Crystal:Crystal_HC18-U_Vertical -> Crystal:Crystal_HC52-U_Horizontal
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Connections:
- C1 pad 1: (no net) -> +5V
- C1 pad 2: (no net) -> GND
- C10 pad 1: (no net) -> +5V
- C10 pad 2: (no net) -> GND
- C11 pad 1: (no net) -> +5V
- C11 pad 2: (no net) -> GND
- C12 pad 1: (no net) -> +5V
- C12 pad 2: (no net) -> GND
- C13 pad 1: (no net) -> +5V
- C13 pad 2: (no net) -> GND
- C14 pad 1: (no net) -> +5V
- C14 pad 2: (no net) -> GND
- C15 pad 1: (no net) -> +5V
- C15 pad 2: (no net) -> GND
- C16 pad 1: (no net) -> +5V
- C16 pad 2: (no net) -> GND
- C17 pad 1: (no net) -> +5V
- C17 pad 2: (no net) -> GND
- C18 pad 1: (no net) -> +5V
- C18 pad 2: (no net) -> GND
- C19 pad 1: (no net) -> +5V
- C19 pad 2: (no net) -> GND
- C2 pad 1: (no net) -> +5V
- C2 pad 2: (no net) -> GND
- C20 pad 1: (no net) -> +5V
- C20 pad 2: (no net) -> GND
- C21 pad 1: (no net) -> +5V
- C21 pad 2: (no net) -> GND
- C22 pad 1: (no net) -> +5V
- C22 pad 2: (no net) -> GND
- C23 pad 1: (no net) -> +5V
- C23 pad 2: (no net) -> GND
- C24 pad 1: (no net) -> +5V
- C24 pad 2: (no net) -> GND
- C25 pad 1: (no net) -> +5V
- C25 pad 2: (no net) -> GND
- C26 pad 1: (no net) -> +5V
- C26 pad 2: (no net) -> GND
- C27 pad 1: (no net) -> +5V
- C27 pad 2: (no net) -> GND
- C28 pad 1: (no net) -> +5V
- C28 pad 2: (no net) -> GND
- C29 pad 1: (no net) -> +5V
- C29 pad 2: (no net) -> GND
- C3 pad 1: (no net) -> +5V
- C3 pad 2: (no net) -> GND
- C30 pad 1: (no net) -> +5V
- C30 pad 2: (no net) -> GND
- C31 pad 1: (no net) -> +5V
- C31 pad 2: (no net) -> GND
- C32 pad 1: (no net) -> +5V
- C32 pad 2: (no net) -> GND
- C33 pad 1: (no net) -> +5V
- C33 pad 2: (no net) -> GND
- C34 pad 1: (no net) -> +5V
- C34 pad 2: (no net) -> GND
- C35 pad 1: (no net) -> +5V
- C35 pad 2: (no net) -> GND
- C36 pad 1: (no net) -> +5V
- C36 pad 2: (no net) -> GND
- C37 pad 1: (no net) -> +5V
- C37 pad 2: (no net) -> GND
- C38 pad 1: (no net) -> +5V
- C38 pad 2: (no net) -> GND
- C39 pad 1: (no net) -> VERIFY_CR1
- C39 pad 2: (no net) -> GND
- C4 pad 1: (no net) -> +5V
- C4 pad 2: (no net) -> GND
- C40 pad 1: (no net) -> +5V
- C40 pad 2: (no net) -> GND
- C41 pad 1: (no net) -> +5V
- C41 pad 2: (no net) -> GND
- C42 pad 1: (no net) -> +5V
- C42 pad 2: (no net) -> GND
- C43 pad 1: (no net) -> +5V
- C43 pad 2: (no net) -> GND
- C44 pad 1: (no net) -> +5V
- C44 pad 2: (no net) -> GND
- C45 pad 1: (no net) -> +5V
- C45 pad 2: (no net) -> GND
- C46 pad 1: (no net) -> +5V
- C46 pad 2: (no net) -> GND
- C47 pad 1: (no net) -> +5V
- C47 pad 2: (no net) -> GND
- C48 pad 1: (no net) -> +5V
- C48 pad 2: (no net) -> GND
- C49 pad 1: (no net) -> +5V
- C49 pad 2: (no net) -> GND
- C5 pad 1: (no net) -> +5V
- C5 pad 2: (no net) -> GND
- C50 pad 1: (no net) -> +5V
- C50 pad 2: (no net) -> GND
- C51 pad 1: (no net) -> +5V
- C51 pad 2: (no net) -> GND
- C52 pad 1: (no net) -> +5V
- C52 pad 2: (no net) -> GND
- C53 pad 1: (no net) -> +5V
- C53 pad 2: (no net) -> GND
- C54 pad 1: (no net) -> +5V
- C54 pad 2: (no net) -> GND
- C6 pad 1: (no net) -> +5V
- C6 pad 2: (no net) -> GND
- C7 pad 1: (no net) -> +5V
- C7 pad 2: (no net) -> GND
- C8 pad 1: (no net) -> +5V
- C8 pad 2: (no net) -> GND
- C9 pad 1: (no net) -> +5V
- C9 pad 2: (no net) -> GND
- CR1 pad 1: (no net) -> +5V
- CR1 pad 2: (no net) -> VERIFY_CR1
- DSW1 pad 1: (no net) -> /Sys.Reset
- DSW1 pad 10: (no net) -> GND
- DSW1 pad 11: (no net) -> GND
- DSW1 pad 12: (no net) -> GND
- DSW1 pad 13: (no net) -> GND
- DSW1 pad 14: (no net) -> GND
- DSW1 pad 15: (no net) -> GND
- DSW1 pad 16: (no net) -> GND
- DSW1 pad 2: (no net) -> /SW_3
- DSW1 pad 3: (no net) -> /SW_2
- DSW1 pad 4: (no net) -> /SW_1
- DSW1 pad 5: (no net) -> /SW_R
- DSW1 pad 6: (no net) -> /SW_H
- DSW1 pad 7: (no net) -> /SW_I
- DSW1 pad 8: (no net) -> /SW_O
- DSW1 pad 9: (no net) -> GND
- J1 pad 1: (no net) -> GND
- J1 pad 10: (no net) -> unconnected-(J1-Pad10)
- J1 pad 11: (no net) -> /Sys.~{A_{1}}
- J1 pad 12: (no net) -> /Sys.~{RDIN}
- J1 pad 13: (no net) -> /Sys.~{A_{2}}
- J1 pad 14: (no net) -> /Sys.~{WTIN}
- J1 pad 15: (no net) -> /Sys.~{A_{3}}
- J1 pad 16: (no net) -> /Sys.~{DRDY}
- J1 pad 17: (no net) -> /Sys.~{A_{4}}
- J1 pad 18: (no net) -> /Sys.~{RA_{14}}
- J1 pad 19: (no net) -> /Sys.~{A_{5}}
- J1 pad 2: (no net) -> GND
- J1 pad 20: (no net) -> /Sys.~{RA_{12}}
- J1 pad 21: (no net) -> /Sys.~{A_{6}}
- J1 pad 22: (no net) -> /Sys.~{APRE}
- J1 pad 23: (no net) -> /Sys.~{A_{7}}
- J1 pad 24: (no net) -> /Sys.~{RA_{13}}
- J1 pad 25: (no net) -> /Sys.~{A_{8}}
- J1 pad 26: (no net) -> /Sys.~{INR1}
- J1 pad 27: (no net) -> /Sys.~{A_{9}}
- J1 pad 28: (no net) -> /Sys.~{INR2}
- J1 pad 29: (no net) -> /Sys.~{A_{10}}
- J1 pad 3: (no net) -> +5V
- J1 pad 30: (no net) -> /Sys.~{INR3}
- J1 pad 31: (no net) -> /Sys.~{PA_{11}}
- J1 pad 32: (no net) -> /Sys.~{INR0}
- J1 pad 33: (no net) -> /Sys.~{PA_{12}}
- J1 pad 34: (no net) -> /Sys.~{RA_{15}}
- J1 pad 35: (no net) -> /Sys.~{PA_{13}}
- J1 pad 36: (no net) -> /Sys.~{CPL_{0}}
- J1 pad 37: (no net) -> /Sys.~{PA_{14}}
- J1 pad 38: (no net) -> /Sys.~{CPL_{1}}
- J1 pad 39: (no net) -> /Sys.~{CA_{15}}
- J1 pad 4: (no net) -> +5V
- J1 pad 40: (no net) -> /Sys.~{CPL_{2}}
- J1 pad 41: (no net) -> /Sys.~{D_{0}}
- J1 pad 42: (no net) -> /Sys.~{CPL_{3}}
- J1 pad 43: (no net) -> /Sys.~{D_{1}}
- J1 pad 44: (no net) -> /Sys.~{RA_{11}}
- J1 pad 45: (no net) -> /Sys.~{D_{2}}
- J1 pad 46: (no net) -> /Sys.~{PA_{15}}
- J1 pad 47: (no net) -> /Sys.~{D_{3}}
- J1 pad 48: (no net) -> /Sys.~{PA_{16}}
- J1 pad 49: (no net) -> /Sys.~{D_{4}}
- J1 pad 5: (no net) -> unconnected-(J1-Pad5)
- J1 pad 50: (no net) -> /Sys.~{PA_{17}}
- J1 pad 51: (no net) -> /Sys.~{D_{5}}
- J1 pad 52: (no net) -> /Sys.~{PTR7_oc}
- J1 pad 53: (no net) -> /Sys.~{D_{6}}
- J1 pad 54: (no net) -> /Sys.~{INTREQ}
- J1 pad 55: (no net) -> /Sys.~{D_{7}}
- J1 pad 56: (no net) -> /Sys.~{MemFault}
- J1 pad 57: (no net) -> /Sys.~{ParityTest}
- J1 pad 58: (no net) -> /Sys.~{INTACK}
- J1 pad 59: (no net) -> Net-(J1-Pad59)
- J1 pad 6: (no net) -> +12V
- J1 pad 60: (no net) -> Net-(J1-Pad59)
- J1 pad 61: (no net) -> /Sys.5MHz
- J1 pad 62: (no net) -> Net-(J1-Pad59)
- J1 pad 63: (no net) -> /Sys.Reset
- J1 pad 64: (no net) -> Net-(J1-Pad59)
- J1 pad 65: (no net) -> Net-(J1-Pad59)
- J1 pad 66: (no net) -> Net-(J1-Pad59)
- J1 pad 67: (no net) -> unconnected-(J1-Pad67)
- J1 pad 68: (no net) -> -12V
- J1 pad 69: (no net) -> +5V
- J1 pad 7: (no net) -> unconnected-(J1-Pad7)
- J1 pad 70: (no net) -> +5V
- J1 pad 8: (no net) -> unconnected-(J1-Pad8)
- J1 pad 9: (no net) -> /Sys.~{A_{0}}
- JP1 pad 1: (no net) -> Net-(JP1-Pad1)
- JP1 pad 2: (no net) -> /PTR.~{Q_{7}}
- JP1 pad 3: (no net) -> Net-(JP1-Pad3)
- P10 pad 1: (no net) -> /PTR.Q_{0}
- P10 pad 10: (no net) -> Address.A_{15}
- P10 pad 11: (no net) -> Address.A_{15}
- P10 pad 12: (no net) -> Address.A_{15}
- P10 pad 13: (no net) -> Address.A_{14}
- P10 pad 14: (no net) -> Address.A_{13}
- P10 pad 15: (no net) -> Address.A_{12}
- P10 pad 16: (no net) -> Address.A_{11}
- P10 pad 2: (no net) -> /PTR.Q_{1}
- P10 pad 3: (no net) -> /PTR.Q_{2}
- P10 pad 4: (no net) -> /PTR.Q_{3}
- P10 pad 5: (no net) -> /PTR.Q_{4}
- P10 pad 6: (no net) -> /PTR.Q_{5}
- P10 pad 7: (no net) -> /PTR.Q_{6}
- P10 pad 8: (no net) -> /PTR.Q_{7}
- P10 pad 9: (no net) -> unconnected-(P10-Pad9)
- P2 pad 1: (no net) -> unconnected-(P2-Pad1)
- P2 pad 10: (no net) -> GND
- P2 pad 11: (no net) -> /DMA.~{Enable}
- P2 pad 12: (no net) -> GND
- P2 pad 13: (no net) -> Net-(P2-Pad13)
- P2 pad 14: (no net) -> GND
- P2 pad 15: (no net) -> /DMA.~{BusReadReady}
- P2 pad 16: (no net) -> GND
- P2 pad 17: (no net) -> /DMA.~{BusWriteOE}
- P2 pad 18: (no net) -> GND
- P2 pad 19: (no net) -> /DMA.~{StartCycle}
- P2 pad 2: (no net) -> GND
- P2 pad 20: (no net) -> GND
- P2 pad 21: (no net) -> /DMA.Write
- P2 pad 22: (no net) -> GND
- P2 pad 23: (no net) -> /DMA.~{INTRequest}
- P2 pad 24: (no net) -> GND
- P2 pad 25: (no net) -> /DMA.~{Request}
- P2 pad 26: (no net) -> GND
- P2 pad 3: (no net) -> /DMA.~{AddressControl}
- P2 pad 4: (no net) -> GND
- P2 pad 5: (no net) -> Net-(P2-Pad5)
- P2 pad 6: (no net) -> GND
- P2 pad 7: (no net) -> Net-(P2-Pad7)
- P2 pad 8: (no net) -> GND
- P2 pad 9: (no net) -> /DMA.~{End}
- P3 pad 1: (no net) -> FP.~{HALT}
- P3 pad 10: (no net) -> GND
- P3 pad 11: (no net) -> Net-(P3-Pad11)
- P3 pad 12: (no net) -> GND
- P3 pad 13: (no net) -> Net-(P3-Pad13)
- P3 pad 14: (no net) -> GND
- P3 pad 15: (no net) -> /SW_2
- P3 pad 16: (no net) -> +5V
- P3 pad 17: (no net) -> /~{ResetFlag}
- P3 pad 18: (no net) -> +5V
- P3 pad 19: (no net) -> Net-(P3-Pad19)
- P3 pad 2: (no net) -> unconnected-(P3-Pad2)
- P3 pad 20: (no net) -> +5V
- P3 pad 21: (no net) -> Net-(P3-Pad21)
- P3 pad 22: (no net) -> +5V
- P3 pad 23: (no net) -> Net-(P3-Pad23)
- P3 pad 24: (no net) -> +5V
- P3 pad 25: (no net) -> FP.RTI
- P3 pad 26: (no net) -> +5V
- P3 pad 3: (no net) -> FP.~{RUN}
- P3 pad 4: (no net) -> /R4_7
- P3 pad 5: (no net) -> Net-(P3-Pad5)
- P3 pad 6: (no net) -> Net-(P3-Pad6)
- P3 pad 7: (no net) -> /SW_O
- P3 pad 8: (no net) -> GND
- P3 pad 9: (no net) -> Net-(P3-Pad9)
- P4 pad 1: (no net) -> GND
- P4 pad 10: (no net) -> DataF.D_{4}
- P4 pad 11: (no net) -> DataF.D_{5}
- P4 pad 12: (no net) -> DataF.D_{6}
- P4 pad 13: (no net) -> DataF.D_{7}
- P4 pad 14: (no net) -> Net-(P4-Pad14)
- P4 pad 15: (no net) -> GND
- P4 pad 16: (no net) -> GND
- P4 pad 2: (no net) -> GND
- P4 pad 3: (no net) -> DataF.D_{0}
- P4 pad 4: (no net) -> DataF.D_{1}
- P4 pad 5: (no net) -> DataF.D_{2}
- P4 pad 6: (no net) -> DataF.D_{3}
- P4 pad 7: (no net) -> /P4_7
- P4 pad 8: (no net) -> +5V
- P4 pad 9: (no net) -> +5V
- P5 pad 1: (no net) -> /MWR.H0_{6}
- P5 pad 10: (no net) -> /MWR.H0_{1}
- P5 pad 11: (no net) -> GND
- P5 pad 12: (no net) -> /MWR.H0_{0}
- P5 pad 13: (no net) -> GND
- P5 pad 14: (no net) -> /MWR.B5_{7}
- P5 pad 15: (no net) -> GND
- P5 pad 16: (no net) -> /MWR.B5_{6}
- P5 pad 17: (no net) -> GND
- P5 pad 18: (no net) -> /MWR.B5_{5}
- P5 pad 19: (no net) -> GND
- P5 pad 2: (no net) -> /MWR.H0_{5}
- P5 pad 20: (no net) -> /MWR.B5_{4}
- P5 pad 21: (no net) -> GND
- P5 pad 22: (no net) -> /MWR.B5_{3}
- P5 pad 23: (no net) -> GND
- P5 pad 24: (no net) -> /MWR.B5_{2}
- P5 pad 25: (no net) -> GND
- P5 pad 26: (no net) -> /MWR.B5_{1}
- P5 pad 27: (no net) -> GND
- P5 pad 28: (no net) -> /MWR.B5_{0}
- P5 pad 29: (no net) -> GND
- P5 pad 3: (no net) -> /MWR.H0_{7}
- P5 pad 30: (no net) -> /MWR.C4_{7}
- P5 pad 31: (no net) -> GND
- P5 pad 32: (no net) -> /MWR.C4_{6}
- P5 pad 33: (no net) -> GND
- P5 pad 34: (no net) -> /MWR.C4_{5}
- P5 pad 35: (no net) -> GND
- P5 pad 36: (no net) -> /MWR.C4_{4}
- P5 pad 37: (no net) -> GND
- P5 pad 38: (no net) -> /MWR.C4_{3}
- P5 pad 39: (no net) -> GND
- P5 pad 4: (no net) -> /MWR.H0_{4}
- P5 pad 40: (no net) -> /MWR.C4_{2}
- P5 pad 41: (no net) -> GND
- P5 pad 42: (no net) -> /MWR.C4_{1}
- P5 pad 43: (no net) -> GND
- P5 pad 44: (no net) -> /MWR.C4_{0}
- P5 pad 45: (no net) -> GND
- P5 pad 46: (no net) -> /MWR.F1_{7}
- P5 pad 47: (no net) -> GND
- P5 pad 48: (no net) -> /MWR.F1_{6}
- P5 pad 49: (no net) -> /MWR.F1_{4}
- P5 pad 5: (no net) -> GND
- P5 pad 50: (no net) -> /MWR.F1_{5}
- P5 pad 6: (no net) -> /MWR.H0_{3}
- P5 pad 7: (no net) -> GND
- P5 pad 8: (no net) -> /MWR.H0_{2}
- P5 pad 9: (no net) -> GND
- P6 pad 1: (no net) -> /MWR.F1_{2}
- P6 pad 10: (no net) -> /MWR.A6_{5}
- P6 pad 11: (no net) -> GND
- P6 pad 12: (no net) -> /MWR.A6_{4}
- P6 pad 13: (no net) -> GND
- P6 pad 14: (no net) -> /MWR.A6_{3}
- P6 pad 15: (no net) -> GND
- P6 pad 16: (no net) -> /MWR.A6_{2}
- P6 pad 17: (no net) -> GND
- P6 pad 18: (no net) -> /MWR.A6_{1}
- P6 pad 19: (no net) -> GND
- P6 pad 2: (no net) -> /MWR.F1_{1}
- P6 pad 20: (no net) -> /MWR.A6_{0}
- P6 pad 21: (no net) -> GND
- P6 pad 22: (no net) -> /MWR.D3_{7}
- P6 pad 23: (no net) -> GND
- P6 pad 24: (no net) -> /MWR.D3_{6}
- P6 pad 25: (no net) -> GND
- P6 pad 26: (no net) -> /MWR.D3_{5}
- P6 pad 27: (no net) -> GND
- P6 pad 28: (no net) -> /MWR.D3_{4}
- P6 pad 29: (no net) -> GND
- P6 pad 3: (no net) -> /MWR.F1_{3}
- P6 pad 30: (no net) -> /MWR.D3_{3}
- P6 pad 31: (no net) -> GND
- P6 pad 32: (no net) -> /MWR.D3_{2}
- P6 pad 33: (no net) -> GND
- P6 pad 34: (no net) -> /MWR.D3_{1}
- P6 pad 35: (no net) -> GND
- P6 pad 36: (no net) -> /MWR.D3_{0}
- P6 pad 37: (no net) -> GND
- P6 pad 38: (no net) -> /MWR.E2_{7}
- P6 pad 39: (no net) -> GND
- P6 pad 4: (no net) -> /MWR.F1_{0}
- P6 pad 40: (no net) -> /MWR.E2_{6}
- P6 pad 41: (no net) -> GND
- P6 pad 42: (no net) -> /MWR.E2_{5}
- P6 pad 43: (no net) -> GND
- P6 pad 44: (no net) -> /MWR.E2_{4}
- P6 pad 45: (no net) -> GND
- P6 pad 46: (no net) -> /MWR.E2_{3}
- P6 pad 47: (no net) -> GND
- P6 pad 48: (no net) -> /MWR.E2_{2}
- P6 pad 49: (no net) -> /MWR.E2_{0}
- P6 pad 5: (no net) -> GND
- P6 pad 50: (no net) -> /MWR.E2_{1}
- P6 pad 6: (no net) -> /MWR.A6_{7}
- P6 pad 7: (no net) -> GND
- P6 pad 8: (no net) -> /MWR.A6_{6}
- P6 pad 9: (no net) -> GND
- P7 pad 1: (no net) -> P7_1
- P7 pad 10: (no net) -> GND
- P7 pad 11: (no net) -> GND
- P7 pad 12: (no net) -> unconnected-(P7-Pad12)
- P7 pad 13: (no net) -> P7_13
- P7 pad 14: (no net) -> /P7_14
- P7 pad 2: (no net) -> P7_2
- P7 pad 3: (no net) -> P7_3
- P7 pad 4: (no net) -> P7_4
- P7 pad 5: (no net) -> P7_5
- P7 pad 6: (no net) -> GND
- P7 pad 7: (no net) -> GND
- P7 pad 8: (no net) -> P7_8
- P7 pad 9: (no net) -> P7_9
- P8 pad 1: (no net) -> GND
- P8 pad 10: (no net) -> MWS.A_{7}
- P8 pad 11: (no net) -> MWS.A_{6}
- P8 pad 12: (no net) -> MWS.A_{2}
- P8 pad 13: (no net) -> MWS.A_{5}
- P8 pad 14: (no net) -> unconnected-(P8-Pad14)
- P8 pad 15: (no net) -> GND
- P8 pad 16: (no net) -> GND
- P8 pad 2: (no net) -> GND
- P8 pad 3: (no net) -> MWS.A_{1}
- P8 pad 4: (no net) -> MWS.A_{0}
- P8 pad 5: (no net) -> MWS.A_{9}
- P8 pad 6: (no net) -> MWS.A_{10}
- P8 pad 7: (no net) -> MWS.A_{4}
- P8 pad 8: (no net) -> MWS.A_{3}
- P8 pad 9: (no net) -> MWS.A_{8}
- R1 pad 1: (no net) -> Net-(P3-Pad6)
- R1 pad 2: (no net) -> FP.~{ABT}
- R10 pad 1: (no net) -> +5V
- R10 pad 2: (no net) -> Net-(R10-Pad2)
- R11 pad 1: (no net) -> +5V
- R11 pad 2: (no net) -> /P7_14
- R12 pad 1: (no net) -> +5V
- R12 pad 2: (no net) -> /P4_7
- R13 pad 1: (no net) -> +5V
- R13 pad 2: (no net) -> Net-(P4-Pad14)
- R14 pad 1: (no net) -> Net-(R14-Pad1)
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Routing:
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
Commit message: Some PoC routing near the bus connector
A checkpoint, i'll try moving chips around in order to optimize tracks
Parts:
- removed the J1 at (369.6, 77.5)
- C39: footprint Capacitor_THT:CP_Axial_L18.0mm_D8.0mm_P25.00mm_Horizontal -> Capacitor_THT:CP_Radial_D8.0mm_P3.50mm
- C52, C53: footprint Capacitor_THT:CP_Axial_L25.0mm_D10.0mm_P30.00mm_Horizontal -> Capacitor_THT:CP_Radial_D8.0mm_P3.50mm
- DSW1: footprint Button_Switch_THT:SW_DIP_SPSTx08_Slide_9.78x22.5mm_W7.62mm_P2.54mm -> Button_Switch_THT:SW_DIP_SPSTx08_Piano_10.8x21.88mm_W7.62mm_P2.54mm
- J1: renamed from REF**; value BUS_EE200 -> Conn_02x36_Top_Bottom
- R7: value 4.7k -> 4.7K; footprint Resistor_THT:R_Array_SIP10 -> Resistor_THT:R_Array_SIP9
- XTAL1: footprint Crystal:Crystal_HC52-U_Horizontal -> Crystal:Crystal_HC18-U_Vertical
- moved R2 42.2 mm to (-2.79, 160.3)
- moved R3 42.2 mm to (-2.79, 156.5)
- moved C54 40.9 mm to (403.4, 147.6)
- moved RN16 37.0 mm to (400.1, 113.0)
- moved C52 26.8 mm to (372.6, 44.5)
- moved C53 25.4 mm to (372.1, 207.0)
- moved U_A4 17.8 mm to (369.6, 67.3)
- moved U_A7 17.8 mm to (369.6, 108.0)
- moved U_A5 17.8 mm to (369.6, 81.3)
- moved U_A8 17.8 mm to (369.6, 121.9)
- moved U_A10 17.8 mm to (369.6, 148.8)
- moved U_A11 17.8 mm to (369.6, 162.2)
- moved U_A12 17.8 mm to (369.6, 175.6)
- moved U_A6 17.8 mm to (369.6, 95.1)
- moved U_A9 17.8 mm to (369.6, 135.3)
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Connections:
- DSW1 pad 1: /Sys.Reset -> GND
- DSW1 pad 10: GND -> /SW_I
- DSW1 pad 11: GND -> /SW_H
- DSW1 pad 12: GND -> /SW_R
- DSW1 pad 13: GND -> /SW_1
- DSW1 pad 14: GND -> /SW_2
- DSW1 pad 15: GND -> /SW_3
- DSW1 pad 16: GND -> /Sys.Reset
- DSW1 pad 2: /SW_3 -> GND
- DSW1 pad 3: /SW_2 -> GND
- DSW1 pad 4: /SW_1 -> GND
- DSW1 pad 5: /SW_R -> GND
- DSW1 pad 6: /SW_H -> GND
- DSW1 pad 7: /SW_I -> GND
- DSW1 pad 8: /SW_O -> GND
- DSW1 pad 9: GND -> /SW_O
- J1 pad 1: (no net) -> GND
- J1 pad 10: (no net) -> /Sys.~{A_{5}}
- J1 pad 11: (no net) -> /Sys.~{A_{6}}
- J1 pad 12: (no net) -> /Sys.~{A_{7}}
- J1 pad 13: (no net) -> /Sys.~{A_{8}}
- J1 pad 14: (no net) -> /Sys.~{A_{9}}
- J1 pad 15: (no net) -> /Sys.~{A_{10}}
- J1 pad 16: (no net) -> /Sys.~{PA_{11}}
- J1 pad 17: (no net) -> /Sys.~{PA_{12}}
- J1 pad 18: (no net) -> /Sys.~{PA_{13}}
- J1 pad 19: (no net) -> /Sys.~{PA_{14}}
- J1 pad 2: (no net) -> +5V
- J1 pad 20: (no net) -> /Sys.~{CA_{15}}
- J1 pad 21: (no net) -> /Sys.~{D_{0}}
- J1 pad 22: (no net) -> /Sys.~{D_{1}}
- J1 pad 23: (no net) -> /Sys.~{D_{2}}
- J1 pad 24: (no net) -> /Sys.~{D_{3}}
- J1 pad 25: (no net) -> /Sys.~{D_{4}}
- J1 pad 26: (no net) -> /Sys.~{D_{5}}
- J1 pad 27: (no net) -> /Sys.~{D_{6}}
- J1 pad 28: (no net) -> /Sys.~{D_{7}}
- J1 pad 29: (no net) -> /Sys.~{ParityTest}
- J1 pad 3: (no net) -> unconnected-(J1-Pad3)
- J1 pad 30: (no net) -> Net-(J1-Pad30)
- J1 pad 31: (no net) -> /Sys.5MHz
- J1 pad 32: (no net) -> /Sys.Reset
- J1 pad 33: (no net) -> Net-(J1-Pad30)
- J1 pad 34: (no net) -> unconnected-(J1-Pad34)
- J1 pad 35: (no net) -> +5V
- J1 pad 36: (no net) -> GND
- J1 pad 37: (no net) -> GND
- J1 pad 38: (no net) -> +5V
- J1 pad 39: (no net) -> +12V
- J1 pad 4: (no net) -> unconnected-(J1-Pad4)
- J1 pad 40: (no net) -> unconnected-(J1-Pad40)
- J1 pad 41: (no net) -> unconnected-(J1-Pad41)
- J1 pad 42: (no net) -> /Sys.~{RDIN}
- J1 pad 43: (no net) -> /Sys.~{WTIN}
- J1 pad 44: (no net) -> /Sys.~{DRDY}
- J1 pad 45: (no net) -> /Sys.~{RA_{14}}
- J1 pad 46: (no net) -> /Sys.~{RA_{12}}
- J1 pad 47: (no net) -> /Sys.~{APRE}
- J1 pad 48: (no net) -> /Sys.~{RA_{13}}
- J1 pad 49: (no net) -> /Sys.~{INR1}
- J1 pad 5: (no net) -> /Sys.~{A_{0}}
- J1 pad 50: (no net) -> /Sys.~{INR2}
- J1 pad 51: (no net) -> /Sys.~{INR3}
- J1 pad 52: (no net) -> /Sys.~{INR0}
- J1 pad 53: (no net) -> /Sys.~{RA_{15}}
- J1 pad 54: (no net) -> /Sys.~{CPL_{0}}
- J1 pad 55: (no net) -> /Sys.~{CPL_{1}}
- J1 pad 56: (no net) -> /Sys.~{CPL_{2}}
- J1 pad 57: (no net) -> /Sys.~{CPL_{3}}
- J1 pad 58: (no net) -> /Sys.~{RA_{11}}
- J1 pad 59: (no net) -> /Sys.~{PA_{15}}
- J1 pad 6: (no net) -> /Sys.~{A_{1}}
- J1 pad 60: (no net) -> /Sys.~{PA_{16}}
- J1 pad 61: (no net) -> /Sys.~{PA_{17}}
- J1 pad 62: (no net) -> /Sys.~{PTR7_oc}
- J1 pad 63: (no net) -> /Sys.~{INTREQ}
- J1 pad 64: (no net) -> /Sys.~{MemFault}
- J1 pad 65: (no net) -> /Sys.~{INTACK}
- J1 pad 66: (no net) -> Net-(J1-Pad30)
- J1 pad 67: (no net) -> Net-(J1-Pad30)
- J1 pad 68: (no net) -> Net-(J1-Pad30)
- J1 pad 69: (no net) -> Net-(J1-Pad30)
- J1 pad 7: (no net) -> /Sys.~{A_{2}}
- J1 pad 70: (no net) -> -12V
- J1 pad 71: (no net) -> +5V
- J1 pad 72: (no net) -> GND
- J1 pad 8: (no net) -> /Sys.~{A_{3}}
- J1 pad 9: (no net) -> /Sys.~{A_{4}}
- P7 pad 14: /P7_14 -> unconnected-(P7-Pad14)
- P7 pad 9: P7_9 -> unconnected-(P7-Pad9)
- R11 pad 2: /P7_14 -> Net-(R11-Pad2)
- R7 pad 2: P7_3 -> unconnected-(R7-Pad2)
- R7 pad 3: /SW_R -> /SW_3
- R7 pad 4: /SW_H -> /SW_1
- R7 pad 5: /SW_I -> /SW_R
- R7 pad 6: /SW_3 -> /SW_H
- R7 pad 7: /SW_1 -> /SW_I
- R7 pad 9: P7_9 -> unconnected-(R7-Pad9)
- U_F5 pad 12: MW.B5_{4} -> MW.B5_{2}
- U_F5 pad 13: /MWR.B5_{4} -> /MWR.B5_{2}
- U_F5 pad 14: /MWR.B5_{5} -> /MWR.B5_{3}
- U_F5 pad 15: MW.B5_{5} -> MW.B5_{3}
- U_F5 pad 6: MW.B5_{2} -> MW.B5_{4}
- U_F5 pad 7: /MWR.B5_{2} -> /MWR.B5_{4}
- U_F5 pad 8: /MWR.B5_{3} -> /MWR.B5_{5}
- U_F5 pad 9: MW.B5_{3} -> MW.B5_{5}
- U_H5 pad 12: MW.C4_{4} -> MW.C4_{2}
- U_H5 pad 13: /MWR.C4_{4} -> /MWR.C4_{2}
- U_H5 pad 14: /MWR.C4_{5} -> /MWR.C4_{3}
- U_H5 pad 15: MW.C4_{5} -> MW.C4_{3}
- U_H5 pad 6: MW.C4_{2} -> MW.C4_{4}
- U_H5 pad 7: /MWR.C4_{2} -> /MWR.C4_{4}
- U_H5 pad 8: /MWR.C4_{3} -> /MWR.C4_{5}
- U_H5 pad 9: MW.C4_{3} -> MW.C4_{5}
- U_J5 pad 12: MW.F1_{4} -> MW.F1_{2}
- U_J5 pad 13: /MWR.F1_{4} -> /MWR.F1_{2}
- U_J5 pad 14: /MWR.F1_{5} -> /MWR.F1_{3}
- U_J5 pad 15: MW.F1_{5} -> MW.F1_{3}
- U_J5 pad 6: MW.F1_{2} -> MW.F1_{4}
- U_J5 pad 7: /MWR.F1_{2} -> /MWR.F1_{4}
- U_J5 pad 8: /MWR.F1_{3} -> /MWR.F1_{5}
- U_J5 pad 9: MW.F1_{3} -> MW.F1_{5}
- U_J6 pad 10: SEQ.~{OE} -> unconnected-(U_J6-Pad10)
- U_J6 pad 11: P7_3 -> GND
- U_J7 pad 22: SEQ.~{OE} -> GND
- U_K5 pad 12: MW.A6_{4} -> MW.A6_{2}
- U_K5 pad 13: /MWR.A6_{4} -> /MWR.A6_{2}
- U_K5 pad 14: /MWR.A6_{5} -> /MWR.A6_{3}
- U_K5 pad 15: MW.A6_{5} -> MW.A6_{3}
- U_K5 pad 6: MW.A6_{2} -> MW.A6_{4}
- U_K5 pad 7: /MWR.A6_{2} -> /MWR.A6_{4}
- U_K5 pad 8: /MWR.A6_{3} -> /MWR.A6_{5}
- U_K5 pad 9: MW.A6_{3} -> MW.A6_{5}
- U_K7 pad 22: SEQ.~{OE} -> GND
- U_L5 pad 12: MW.D3_{4} -> MW.D3_{2}
- U_L5 pad 13: /MWR.D3_{4} -> /MWR.D3_{2}
- U_L5 pad 14: /MWR.D3_{5} -> /MWR.D3_{3}
- U_L5 pad 15: MW.D3_{5} -> MW.D3_{3}
- U_L5 pad 6: MW.D3_{2} -> MW.D3_{4}
- U_L5 pad 7: /MWR.D3_{2} -> /MWR.D3_{4}
- U_L5 pad 8: /MWR.D3_{3} -> /MWR.D3_{5}
- U_L5 pad 9: MW.D3_{3} -> MW.D3_{5}
- U_L6 pad 9: P7_9 -> /~{MAPROM_SEL}
- U_L9 pad 22: SEQ.~{OE} -> GND
- U_M5 pad 12: MW.E2_{4} -> MW.E2_{2}
- U_M5 pad 13: /MWR.E2_{4} -> /MWR.E2_{2}
- U_M5 pad 14: /MWR.E2_{5} -> /MWR.E2_{3}
- U_M5 pad 15: MW.E2_{5} -> MW.E2_{3}
- U_M5 pad 6: MW.E2_{2} -> MW.E2_{4}
- U_M5 pad 7: /MWR.E2_{2} -> /MWR.E2_{4}
- U_M5 pad 8: /MWR.E2_{3} -> /MWR.E2_{5}
- U_M5 pad 9: MW.E2_{3} -> MW.E2_{5}
- U_M6 pad 11: MW.E2_{3} -> MW.E2_{2}
- U_M6 pad 12: DataP.D_{7} -> DataP.D_{5}
- U_M6 pad 13: MW.E2_{2} -> MW.E2_{3}
- U_M6 pad 14: DataP.D_{6} -> DataP.D_{4}
- U_M6 pad 16: DataP.D_{5} -> DataP.D_{6}
- U_M6 pad 18: DataP.D_{4} -> DataP.D_{7}
- U_M6 pad 2: MW.E2_{4} -> MW.E2_{7}
- U_M6 pad 4: MW.E2_{5} -> MW.E2_{6}
- U_M6 pad 6: MW.E2_{6} -> MW.E2_{4}
- U_M6 pad 7: DataP.D_{2} -> DataP.D_{3}
- U_M6 pad 8: MW.E2_{7} -> MW.E2_{5}
- U_M6 pad 9: DataP.D_{3} -> DataP.D_{2}
- U_M7 pad 11: /SW_1 -> /SW_3
- U_M7 pad 12: DataP.D_{0} -> DataP.D_{2}
- U_M7 pad 13: /SW_2 -> /~{FPC_SW_4}
- U_M7 pad 14: DataP.D_{1} -> DataP.D_{3}
- U_M7 pad 15: /SW_3 -> /SW_2
- U_M7 pad 16: DataP.D_{2} -> DataP.D_{1}
- U_M7 pad 17: /~{FPC_SW_4} -> /SW_1
- U_M7 pad 18: DataP.D_{3} -> DataP.D_{0}
- U_M7 pad 2: /SW_R -> /~{RT_INT}
- U_M7 pad 3: DataP.D_{3} -> DataP.D_{0}
- U_M7 pad 4: /SW_H -> /SW_I
- U_M7 pad 5: DataP.D_{2} -> DataP.D_{1}
- U_M7 pad 6: /SW_I -> /SW_R
- U_M7 pad 7: DataP.D_{1} -> DataP.D_{3}
- U_M7 pad 8: /~{RT_INT} -> /SW_H
- U_M7 pad 9: DataP.D_{0} -> DataP.D_{2}
- U_MWE2 pad 18: /P7_14 -> Net-(R11-Pad2)
- U_MWF2 pad 18: /P7_14 -> Net-(R11-Pad2)
- U_MWH2 pad 18: /P7_14 -> Net-(R11-Pad2)
- U_MWJ2 pad 18: /P7_14 -> Net-(R11-Pad2)
- U_MWK2 pad 18: /P7_14 -> Net-(R11-Pad2)
- U_MWL2 pad 18: /P7_14 -> Net-(R11-Pad2)
- U_MWM2 pad 18: /P7_14 -> Net-(R11-Pad2)
Routing:
- net /Page.B_{2}: track 0.00 -> 213.8 mm
- net /Page.B_{0}: track 0.00 -> 189.5 mm
- net /Page.B_{1}: track 0.00 -> 185.6 mm
- net Net-(R11-Pad2): track 0.00 -> 174.0 mm
- net /P7_14: track 174.0 -> 0.00 mm
- net /R4_7: track 0.00 -> 130.7 mm
- net /SW_O: track 0.00 -> 96.2 mm
- net /DMA.~{INTRequest}: track 0.00 -> 87.3 mm
- net GND: track 704.7 -> 788.8 mm
- net /SW_1: track 0.00 -> 74.9 mm
- net /Sys.~{WTIN}: track 0.00 -> 70.0 mm, vias 0 -> 1
- net Net-(P3-Pad19): track 0.00 -> 69.5 mm
- net /Sys.~{RA_{13}}: track 0.00 -> 68.7 mm, vias 0 -> 1
- net /SW_3: track 0.00 -> 67.6 mm
- net /Sys.~{APRE}: track 0.00 -> 66.3 mm, vias 0 -> 1
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
Commit message: Routing WIP
Checkpoint
Parts:
- moved U_A10 13.6 mm to (369.8, 135.1)
- moved U_A6 13.4 mm to (369.6, 108.5)
- moved U_A9 13.3 mm to (369.6, 148.6)
- moved U_A7 12.7 mm to (369.6, 95.3)
- moved RN16 7.37 mm to (392.7, 113.0)
Connections:
- U_A3 pad 10: /Sys.~{RA_{14}} -> /Sys.~{RA_{12}}
- U_A3 pad 11: Address.A_{14} -> Address.A_{12}
- U_A3 pad 8: /Sys.~{RA_{12}} -> /Sys.~{RA_{14}}
- U_A3 pad 9: Address.A_{12} -> Address.A_{14}
- U_A6 pad 11: Address.A_{8} -> unconnected-(U_A6-Pad11)
- U_A6 pad 12: DataP.D_{4} -> DataP.D_{7}
- U_A6 pad 14: DataP.D_{5} -> DataP.D_{6}
- U_A6 pad 16: DataP.D_{6} -> DataP.D_{5}
- U_A6 pad 18: DataP.D_{7} -> DataP.D_{4}
- U_A6 pad 2: /CPL_{3} -> /CPL_{0}
- U_A6 pad 4: /CPL_{2} -> /CPL_{1}
- U_A6 pad 6: /CPL_{1} -> /CPL_{2}
- U_A6 pad 8: /CPL_{0} -> /CPL_{3}
- U_A7 pad 12: DataP.D_{4} -> DataP.D_{7}
- U_A7 pad 14: DataP.D_{5} -> DataP.D_{6}
- U_A7 pad 16: DataP.D_{6} -> DataP.D_{5}
- U_A7 pad 18: DataP.D_{7} -> DataP.D_{4}
- U_A7 pad 2: /Sys.~{INR3} -> /Sys.~{INR0}
- U_A7 pad 4: /Sys.~{INR2} -> /Sys.~{INR1}
- U_A7 pad 6: /Sys.~{INR1} -> /Sys.~{INR2}
- U_A7 pad 8: /Sys.~{INR0} -> /Sys.~{INR3}
- U_A8 pad 12: /Sys.~{CPL_{0}} -> /Sys.~{CPL_{3}}
- U_A8 pad 14: /Sys.~{CPL_{1}} -> /Sys.~{CPL_{2}}
- U_A8 pad 16: /Sys.~{CPL_{2}} -> /Sys.~{CPL_{1}}
- U_A8 pad 18: /Sys.~{CPL_{3}} -> /Sys.~{CPL_{0}}
- U_A8 pad 2: /CPL_{3} -> /CPL_{0}
- U_A8 pad 4: /CPL_{2} -> /CPL_{1}
- U_A8 pad 6: /CPL_{1} -> /CPL_{2}
- U_A8 pad 8: /CPL_{0} -> /CPL_{3}
- U_A9 pad 12: DataP.D_{6} -> DataP.D_{7}
- U_A9 pad 14: DataP.D_{7} -> DataP.D_{6}
- U_A9 pad 6: Net-(U_A10-Pad6) -> /PTR.Q_{6}
- U_A9 pad 8: /PTR.Q_{6} -> Net-(U_A10-Pad6)
Routing:
- net /BUS_TIMEOUT: track 0.00 -> 184.1 mm
- net Address.A_{13}: track 0.00 -> 67.2 mm
- net /Sys.~{D_{1}}: track 0.00 -> 60.0 mm
- net /Sys.~{D_{5}}: track 0.00 -> 55.3 mm
- net /Sys.~{D_{0}}: track 0.00 -> 53.0 mm
- net /Sys.~{D_{4}}: track 0.00 -> 52.5 mm
- net Address.A_{14}: track 0.00 -> 48.5 mm
- net /Sys.~{PA_{11}}: track 0.00 -> 47.0 mm
- net /Sys.~{A_{8}}: track 0.00 -> 44.7 mm
- net Address.A_{12}: track 0.00 -> 43.6 mm
- net DataP.D_{3}: track 23.9 -> 66.1 mm
- net /Sys.~{PA_{12}}: track 0.00 -> 38.3 mm
- net /Sys.~{A_{9}}: track 0.00 -> 37.9 mm
- net /Sys.~{INR3}: track 0.00 -> 37.8 mm, vias 0 -> 1
- net /Sys.~{PA_{17}}: track 0.00 -> 35.0 mm
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