File: FrontPanel/FrontPanel.kicad_pcb (KiCad board)
At the start: 2 copper layers, 266.7 x 88.9 mm, 70 parts, among them J1 CPU, J2 Backplane, U1 74LS38, U2 74LS38, U3 74LS123, U4 NE555P

Commit message: FrontPanel: Parts placement
Placed all the parts close to original layout.
Parts:
- added J3: Conn_01x05_Male, Connector_PinHeader_2.54mm:PinHeader_1x05_P2.54mm_Vertical, F.Cu at (360.3, 119.5)
- added REF**: MountingHole_2.5mm, MountingHole:MountingHole_2.5mm, F.Cu at (361.9, 162.6)
- added REF**: MountingHole_2.5mm, MountingHole:MountingHole_2.5mm, F.Cu at (108.0, 161.3)
- C1, C2, C3: footprint Capacitor_THT:CP_Radial_D8.0mm_P3.50mm -> Capacitor_THT:CP_Axial_L18.0mm_D6.5mm_P25.00mm_Horizontal
- D30, D31, D32, D33, D34, D35: footprint Diode_THT:D_A-405_P7.62mm_Horizontal -> Diode_THT:D_A-405_P10.16mm_Horizontal
- moved D31 415.8 mm to (327.4, 162.9), turned to 90 degrees
- moved R23 412.2 mm to (319.7, 165.4), turned to 90 degrees
- moved R1 387.7 mm to (278.6, 133.3)
- moved R6 385.0 mm to (265.6, 141.0), turned to -90 degrees
- moved R3 383.5 mm to (299.5, 140.7), turned to 90 degrees
- moved D33 380.7 mm to (293.6, 157.4), turned to 180 degrees
- moved D32 375.3 mm to (312.4, 162.9), turned to 90 degrees
- moved R2 364.0 mm to (292.9, 140.6), turned to 90 degrees
- moved R5 361.5 mm to (278.6, 136.8)
- moved C3 361.4 mm to (299.4, 150.1), turned to 180 degrees
- moved R8 342.5 mm to (233.0, 142.2), turned to -90 degrees
- moved C4 338.3 mm to (250.2, 157.4), turned to 90 degrees
- moved D35 335.3 mm to (278.7, 140.8)
- moved D34 334.3 mm to (251.8, 140.7), turned to 180 degrees
- moved R11 333.3 mm to (236.2, 142.2), turned to -90 degrees
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Connections:
- net Net-(U1-Pad10) renamed /R/F
- net Net-(U2-Pad10) renamed /Select
- net Net-(U2-Pad4) renamed /OpSys
- net Net-(U3-Pad1) renamed /Reset
- C1 pad 2: GND -> GNDD
- J1 pad 10: GND -> GNDD
- J1 pad 12: GND -> GNDD
- J1 pad 14: GND -> GNDD
- J1 pad 8: GND -> GNDD
- R10 pad 2: GND -> GNDD
- R4 pad 1: GND -> GNDD
- R4 pad 2: Earth -> GND
- U1 pad 7: GND -> GNDD

Commit message: FrontPanel: Fixed J2 bottom pinout
Fix swapped 5V and GND, verified with the photo
Parts:
- moved J1 19.6 mm to (195.5, 86.0)
- moved J2 16.9 mm to (287.4, 86.0)
- moved C4 2.29 mm to (247.9, 157.4)
- moved D34 0.89 mm to (251.0, 140.7)
Connections:
- J2 pad 10: GND -> +5V
- J2 pad 12: GND -> +5V
- J2 pad 14: GND -> +5V
- J2 pad 16: GND -> +5V
- J2 pad 18: GND -> +5V
- J2 pad 2: GND -> +5V
- J2 pad 20: GND -> +5V
- J2 pad 22: GND -> +5V
- J2 pad 24: GND -> +5V
- J2 pad 28: +5V -> GND
- J2 pad 30: +5V -> GND
- J2 pad 32: +5V -> GND
- J2 pad 34: +5V -> GND
- J2 pad 36: +5V -> GND
- J2 pad 38: +5V -> GND
- J2 pad 4: unconnected-(J2-Pad4) -> +5V
- J2 pad 40: +5V -> GND
- J2 pad 42: +5V -> GND
- J2 pad 44: +5V -> GND
- J2 pad 46: +5V -> GND
- J2 pad 48: +5V -> unconnected-(J2-Pad48)
- J2 pad 50: +5V -> GND
- J2 pad 6: GND -> +5V
- J2 pad 8: GND -> +5V
Routing:
- net GND: track 0.00 -> 316.0 mm
- net /R/F: track 0.00 -> 207.4 mm
- net +5V: track 0.00 -> 163.5 mm
- net GNDD: track 0.00 -> 48.8 mm
- net Net-(D31-Pad2): track 0.00 -> 47.0 mm
- net Net-(D14-Pad1): track 0.00 -> 45.1 mm
- net Net-(D9-Pad1): track 0.00 -> 35.8 mm
- net Net-(D17-Pad1): track 0.00 -> 30.4 mm
- net Net-(D1-Pad1): track 0.00 -> 28.6 mm
- net Net-(C4-Pad1): track 0.00 -> 26.2 mm
- net Net-(C4-Pad2): track 0.00 -> 6.95 mm

Commit message: FrontPanel: Complete
Add potentiometer to adjust clock frequency and better connector for buttons.
Complete the layout.
Parts:
- added RV1: 50K, Potentiometer_THT:Potentiometer_Bourns_3299Y_Vertical, F.Cu at (142.2, 102.3)
- D30, D31, D32, D33, D34, D35: value D -> 1N4148
- J3: value Conn_01x05_Male -> MPW-Y; footprint Connector_PinHeader_2.54mm:PinHeader_1x05_P2.54mm_Vertical -> Connector_Phoenix_MSTB:PhoenixContact_MSTBVA_2,5_5-G-5,08_1x05_P5.08mm_Vertical
- R21: value 144K -> 100K
- moved R1 73.6 mm to (347.4, 107.2), turned to -90 degrees
- moved R2 66.8 mm to (350.8, 107.2), turned to -90 degrees
- moved R3 64.1 mm to (354.2, 107.2), turned to -90 degrees
- moved R23 53.8 mm to (344.1, 117.4)
- moved R5 24.0 mm to (255.3, 131.2)
- moved C3 23.3 mm to (287.0, 130.4), turned to -90 degrees
- moved D33 14.7 mm to (280.0, 163.1), turned to 90 degrees
- moved R7 9.92 mm to (204.0, 139.4), turned to -90 degrees
- moved R21 8.10 mm to (122.1, 107.3)
- moved C5 7.65 mm to (131.3, 97.9)
- moved R22 7.65 mm to (131.8, 95.4)
- moved U4 7.65 mm to (118.6, 92.9)
- moved R10 6.10 mm to (198.0, 131.2)
- moved D6 2.55 mm to (335.3, 135.9), turned to 0 degrees
- moved D8 2.55 mm to (335.3, 154.9), turned to 0 degrees
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Connections:
- R21 pad 1: Net-(U4-Pad7) -> Net-(C5-Pad1)
- R21 pad 2: Net-(C5-Pad1) -> Net-(R21-Pad2)
- R22 pad 1: Net-(U4-Pad7) -> Net-(R22-Pad1)
- U4 pad 7: Net-(U4-Pad7) -> Net-(R22-Pad1)
Routing:
- net +5V: track 163.5 -> 526.9 mm
- net GND: track 316.0 -> 499.2 mm
- net /OpSys: track 0.00 -> 180.6 mm, vias 0 -> 1
- net Net-(D8-Pad2): track 0.00 -> 174.8 mm
- net /Select: track 0.00 -> 172.4 mm, vias 0 -> 1
- net Net-(D7-Pad2): track 0.00 -> 150.8 mm
- net Net-(D6-Pad2): track 0.00 -> 148.8 mm
- net Net-(D29-Pad1): track 0.00 -> 136.4 mm
- net Net-(D4-Pad2): track 0.00 -> 124.3 mm
- net /Reset: track 0.00 -> 123.9 mm
- net Net-(D28-Pad1): track 0.00 -> 119.9 mm
- net Net-(D2-Pad2): track 0.00 -> 119.2 mm
- net Net-(D3-Pad2): track 0.00 -> 118.6 mm
- net Net-(D5-Pad2): track 0.00 -> 111.2 mm
- net Net-(D1-Pad2): track 0.00 -> 103.5 mm
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
Commit message: FrontPanel: Add missing mounting holes
Got information on their placement, so put them in
Parts:
- added REF**: MountingHole_2.5mm, MountingHole:MountingHole_2.5mm, F.Cu at (108.0, 104.1)
- added REF**: MountingHole_2.5mm, MountingHole:MountingHole_2.5mm, F.Cu at (361.9, 104.1)
Changed lines of the file:
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@@
   )
   (paper "A3")
+  (title_block
+    (title "Centurion front panel replica")
+    (rev "1.0")
+  )
   (layers
     (0 "F.Cu" signal)
@@
   (net 81 "unconnected-(J2-Pad48)")
   (net 82 "Net-(D25-Pad1)")
+  (footprint "MountingHole:MountingHole_2.5mm" (layer "F.Cu")
+    (at 107.95 104.14)
+    (descr "Mounting Hole 2.5mm, no annular")
+    (tags "mounting hole 2.5mm no annular")
+    (attr exclude_from_pos_files exclude_from_bom)
+    (fp_text reference "REF**" (at 0 -3.5) (layer "F.SilkS") hide
+      (effects (font (size 1 1) (thickness 0.15)))
+    )
+    (fp_text value "MountingHole_2.5mm" (at 0 3.5) (layer "F.Fab")
+      (effects (font (size 1 1) (thickness 0.15)))
+    )
+    (fp_text user "${REFERENCE}" (at 0 0) (layer "F.Fab") hide
+      (effects (font (size 1 1) (thickness 0.15)))
+    )
+    (fp_circle (center 0 0) (end 2.5 0) (layer "Cmts.User") (width 0.15) (fill none))
+    (fp_circle (center 0 0) (end 2.75 0) (layer "F.CrtYd") (width 0.05) (fill none))
+    (pad "" np_thru_hole circle (at 0 0) (size 2.5 2.5) (drill 2.5) (layers F&B.Cu *.Mask))
+  )
   (footprint "Resistor_THT:R_Axial_DIN0207_L6.3mm_D2.5mm_P10.16mm_Horizontal" (layer "F.Cu")
     (at 160.02 140.589)
@@
     )
   )
+  (footprint "MountingHole:MountingHole_2.5mm" (layer "F.Cu")
+    (at 361.949999 104.14)
+    (descr "Mounting Hole 2.5mm, no annular")
+    (tags "mounting hole 2.5mm no annular")
+    (attr exclude_from_pos_files exclude_from_bom)
+    (fp_text reference "REF**" (at 0 -3.5) (layer "F.SilkS") hide
+      (effects (font (size 1 1) (thickness 0.15)))
+    )
+    (fp_text value "MountingHole_2.5mm" (at 0 3.5) (layer "F.Fab")
+      (effects (font (size 1 1) (thickness 0.15)))
+    )
+    (fp_text user "${REFERENCE}" (at 0 0) (layer "F.Fab") hide
+      (effects (font (size 1 1) (thickness 0.15)))
+    )
+    (fp_circle (center 0 0) (end 2.5 0) (layer "Cmts.User") (width 0.15) (fill none))
+    (fp_circle (center 0 0) (end 2.75 0) (layer "F.CrtYd") (width 0.05) (fill none))
+    (pad "" np_thru_hole circle (at 0 0) (size 2.5 2.5) (drill 2.5) (layers F&B.Cu *.Mask))
+  )
   (footprint "Resistor_THT:R_Axial_DIN0207_L6.3mm_D2.5mm_P10.16mm_Horizontal" (layer "F.Cu")
     (at 236.22 144.78 -90)
@@
     (pts (xy 304.8 167.64) (xy 273.05 167.64))
     (height -12.7)
-    (gr_text "31.7500 mm" (at 288.925 179.19) (layer "Dwgs.User")
+    (gr_text "1.2500 in" (at 288.925 179.19) (layer "Dwgs.User")
       (effects (font (size 1 1) (thickness 0.15)))
     )
@@
     (pts (xy 146.05 167.64) (xy 114.3 167.64))
     (height -12.7)
-    (gr_text "31.7500 mm" (at 130.175 179.19) (layer "Dwgs.User")
+    (gr_text "1.2500 in" (at 130.175 179.19) (layer "Dwgs.User")
       (effects (font (size 1 1) (thickness 0.15)))
     )
@@
     (pts (xy 336.55 167.64) (xy 304.8 167.64))
     (height -12.7)
-    (gr_text "31.7500 mm" (at 320.675 179.19) (layer "Dwgs.User")
+    (gr_text "1.2500 in" (at 320.675 179.19) (layer "Dwgs.User")
       (effects (font (size 1 1) (thickness 0.15)))
     )
@@
     (pts (xy 241.3 167.64) (xy 209.55 167.64))
     (height -12.7)
-    (gr_text "31.7500 mm" (at 225.425 179.19) (layer "Dwgs.User")
+    (gr_text "1.2500 in" (at 225.425 179.19) (layer "Dwgs.User")
       (effects (font (size 1 1) (thickness 0.15)))
     )
@@
     (pts (xy 101.6 167.64) (xy 107.95 167.64))
     (height 6.35)
-    (gr_text "6.35 mm" (at 104.775 172.84) (layer "Dwgs.User")
+    (gr_text "0.25 in" (at 104.775 172.84) (layer "Dwgs.User")
       (effects (font (size 1 1) (thickness 0.15)))
     )
@@
     (pts (xy 177.8 167.64) (xy 146.05 167.64))
     (height -12.7)
-    (gr_text "31.7500 mm" (at 161.925 179.19) (layer "Dwgs.User")
+    (gr_text "1.2500 in" (at 161.925 179.19) (layer "Dwgs.User")
       (effects (font (size 1 1) (thickness 0.15)))
     )
@@
     (pts (xy 101.6 145.415) (xy 101.6 135.89))
     (height -11.43)
-    (gr_text "9.525 mm" (at 89.02 140.6525 90) (layer "Dwgs.User")
+    (gr_text "0.375 in" (at 89.02 140.6525 90) (layer "Dwgs.User")
       (effects (font (size 1 1) (thickness 0.15)))
     )
@@
     (pts (xy 101.6 135.89) (xy 101.6 126.365))
     (height -11.43)
-    (gr_text "9.525 mm" (at 89.02 131.1275 90) (layer "Dwgs.User")
+    (gr_text "0.375 in" (at 89.02 131.1275 90) (layer "Dwgs.User")
       (effects (font (size 1 1) (thickness 0.15)))
     )
@@
     (pts (xy 368.3 167.64) (xy 101.6 167.64))
     (height -22.86)
-    (gr_text "266.7 mm" (at 234.95 189.35) (layer "Dwgs.User")
+    (gr_text "10.5 in" (at 234.95 189.35) (layer "Dwgs.User")
       (effects (font (size 1 1) (thickness 0.15)))
     )
@@
     (pts (xy 209.55 167.64) (xy 177.8 167.64))
     (height -12.7)
-    (gr_text "31.7500 mm" (at 193.675 179.19) (layer "Dwgs.User")
+    (gr_text "1.2500 in" (at 193.675 179.19) (layer "Dwgs.User")
       (effects (font (size 1 1) (thickness 0.15)))
     )
@@
     (pts (xy 368.3 167.64) (xy 368.3 78.74))
     (height 16.51)
-    (gr_text "88.9000 mm" (at 383.66 123.19 90) (layer "Dwgs.User")
+    (gr_text "3.5000 in" (at 383.66 123.19 90) (layer "Dwgs.User")
       (effects (font (size 1 1) (thickness 0.15)))
     )
@@
     (pts (xy 273.05 167.64) (xy 241.3 167.64))
     (height -12.7)
-    (gr_text "31.7500 mm" (at 257.175 179.19) (layer "Dwgs.User")
+    (gr_text "1.2500 in" (at 257.175 179.19) (layer "Dwgs.User")
       (effects (font (size 1 1) (thickness 0.15)))
     )
@@
     (pts (xy 368.3 167.64) (xy 336.55 167.64))
     (height -12.7)
-    (gr_text "31.75 mm" (at 352.425 179.19) (layer "Dwgs.User")
+    (gr_text "1.25 in" (at 352.425 179.19) (layer "Dwgs.User")
       (effects (font (size 1 1) (thickness 0.15)))
     )
@@
     (style (thickness 0.1) (arrow_length 1.27) (text_position_mode 0) (extension_height 0.58642) (extension_offset 0.5) keep_text_aligned)
   )
+  (dimension (type aligned) (layer "Dwgs.User")
+    (pts (xy 101.6 78.74) (xy 101.6 104.14))
+    (height 12.7)
+    (gr_text "1.0000 in" (at 87.75 91.44 90) (layer "Dwgs.User")
+      (effects (font (size 1 1) (thickness 0.15)))
+    )
+    (format (units 3) (units_format 1) (precision 4))
+    (style (thickness 0.1) (arrow_length 1.27) (text_position_mode 0) (extension_height 0.58642) (extension_offset 0.5) keep_text_aligned)
+  )

Commit message: FrontPanel: Add copper pour
This board also fills pretty well, so let's do it.
Routing:
- added copper zone on F.Cu, net +5V
- added copper zone on B.Cu, net GND
Changed lines of the file:
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@@
     (pts (xy 304.8 167.64) (xy 273.05 167.64))
     (height -12.7)
-    (gr_text "1.2500 in" (at 288.925 179.19) (layer "Dwgs.User")
+    (gr_text "31.7500 mm" (at 288.925 179.19) (layer "Dwgs.User")
       (effects (font (size 1 1) (thickness 0.15)))
     )
@@
     (pts (xy 146.05 167.64) (xy 114.3 167.64))
     (height -12.7)
-    (gr_text "1.2500 in" (at 130.175 179.19) (layer "Dwgs.User")
+    (gr_text "31.7500 mm" (at 130.175 179.19) (layer "Dwgs.User")
       (effects (font (size 1 1) (thickness 0.15)))
     )
@@
     (pts (xy 336.55 167.64) (xy 304.8 167.64))
     (height -12.7)
-    (gr_text "1.2500 in" (at 320.675 179.19) (layer "Dwgs.User")
+    (gr_text "31.7500 mm" (at 320.675 179.19) (layer "Dwgs.User")
       (effects (font (size 1 1) (thickness 0.15)))
     )
@@
     (pts (xy 241.3 167.64) (xy 209.55 167.64))
     (height -12.7)
-    (gr_text "1.2500 in" (at 225.425 179.19) (layer "Dwgs.User")
+    (gr_text "31.7500 mm" (at 225.425 179.19) (layer "Dwgs.User")
       (effects (font (size 1 1) (thickness 0.15)))
     )
@@
     (pts (xy 101.6 167.64) (xy 107.95 167.64))
     (height 6.35)
-    (gr_text "0.25 in" (at 104.775 172.84) (layer "Dwgs.User")
+    (gr_text "6.35 mm" (at 104.775 172.84) (layer "Dwgs.User")
       (effects (font (size 1 1) (thickness 0.15)))
     )
@@
     (pts (xy 177.8 167.64) (xy 146.05 167.64))
     (height -12.7)
-    (gr_text "1.2500 in" (at 161.925 179.19) (layer "Dwgs.User")
+    (gr_text "31.7500 mm" (at 161.925 179.19) (layer "Dwgs.User")
       (effects (font (size 1 1) (thickness 0.15)))
     )
@@
     (pts (xy 101.6 145.415) (xy 101.6 135.89))
     (height -11.43)
-    (gr_text "0.375 in" (at 89.02 140.6525 90) (layer "Dwgs.User")
+    (gr_text "9.525 mm" (at 89.02 140.6525 90) (layer "Dwgs.User")
       (effects (font (size 1 1) (thickness 0.15)))
     )
@@
     (pts (xy 101.6 135.89) (xy 101.6 126.365))
     (height -11.43)
-    (gr_text "0.375 in" (at 89.02 131.1275 90) (layer "Dwgs.User")
+    (gr_text "9.525 mm" (at 89.02 131.1275 90) (layer "Dwgs.User")
       (effects (font (size 1 1) (thickness 0.15)))
     )
@@
     (pts (xy 368.3 167.64) (xy 101.6 167.64))
     (height -22.86)
-    (gr_text "10.5 in" (at 234.95 189.35) (layer "Dwgs.User")
+    (gr_text "266.7 mm" (at 234.95 189.35) (layer "Dwgs.User")
       (effects (font (size 1 1) (thickness 0.15)))
     )
@@
     (pts (xy 209.55 167.64) (xy 177.8 167.64))
     (height -12.7)
-    (gr_text "1.2500 in" (at 193.675 179.19) (layer "Dwgs.User")
+    (gr_text "31.7500 mm" (at 193.675 179.19) (layer "Dwgs.User")
       (effects (font (size 1 1) (thickness 0.15)))
     )
@@
     (pts (xy 368.3 167.64) (xy 368.3 78.74))
     (height 16.51)
-    (gr_text "3.5000 in" (at 383.66 123.19 90) (layer "Dwgs.User")
+    (gr_text "88.9000 mm" (at 383.66 123.19 90) (layer "Dwgs.User")
       (effects (font (size 1 1) (thickness 0.15)))
     )
@@
     (pts (xy 273.05 167.64) (xy 241.3 167.64))
     (height -12.7)
-    (gr_text "1.2500 in" (at 257.175 179.19) (layer "Dwgs.User")
+    (gr_text "31.7500 mm" (at 257.175 179.19) (layer "Dwgs.User")
       (effects (font (size 1 1) (thickness 0.15)))
     )
@@
     (pts (xy 368.3 167.64) (xy 336.55 167.64))
     (height -12.7)
-    (gr_text "1.25 in" (at 352.425 179.19) (layer "Dwgs.User")
+    (gr_text "31.75 mm" (at 352.425 179.19) (layer "Dwgs.User")
       (effects (font (size 1 1) (thickness 0.15)))
     )
@@
     (pts (xy 101.6 78.74) (xy 101.6 104.14))
     (height 12.7)
-    (gr_text "1.0000 in" (at 87.75 91.44 90) (layer "Dwgs.User")
+    (gr_text "25.4000 mm" (at 87.75 91.44 90) (layer "Dwgs.User")
       (effects (font (size 1 1) (thickness 0.15)))
     )
@@
   (segment (start 142.367 122.555) (end 144.526 120.396) (width 0.3) (layer "F.Cu") (net 82))
   (segment (start 147.325 135.89) (end 147.325 134.244) (width 0.3) (layer "F.Cu") (net 82))
+  (zone (net 0) (net_name "") (layer "F.Cu") (hatch edge 0.508)
+    (connect_pads (clearance 0))
+    (min_thickness 0.254)
+    (keepout (tracks not_allowed) (vias not_allowed) (pads not_allowed) (copperpour not_allowed) (footprints allowed))
+    (fill (thermal_gap 0.508) (thermal_bridge_width 0.508))
+    (polygon
+      (pts
+        (xy 367 109.5)
+        (xy 357 109.5)
+        (xy 357 99)
+        (xy 367 99)
+      )
+    )
+  )
+  (zone (net 1) (net_name "+5V") (layer "F.Cu") (hatch edge 0.508)
+    (connect_pads (clearance 0.508))
+    (min_thickness 0.254) (filled_areas_thickness no)
+    (fill yes (thermal_gap 0.508) (thermal_bridge_width 0.508))
+    (polygon
+      (pts
+        (xy 368.25 78.75)
+        (xy 368.25 127.25)
+        (xy 368.25 128.5)
+        (xy 368.25 147)
+        (xy 347.5 167.5)
+        (xy 122 167.5)
+        (xy 101.5 147)
+        (xy 101.5 145)
+        (xy 101.5 115.25)
+        (xy 101.5 78.75)
+        (xy 112 78.75)
+        (xy 112.5 78.75)
+        (xy 357.25 78.75)
+      )
+    )
+  )
+  (zone (net 0) (net_name "") (layer "F.Cu") (hatch edge 0.508)
+    (connect_pads (clearance 0))
+    (min_thickness 0.254)
+    (keepout (tracks not_allowed) (vias not_allowed) (pads not_allowed) (copperpour not_allowed) (footprints allowed))
+    (fill (thermal_gap 0.508) (thermal_bridge_width 0.508))
+    (polygon
+      (pts
+        (xy 113 109.5)
+        (xy 103 109.5)
+        (xy 103 99)
+        (xy 113 99)
+      )
+    )
+  )
+  (zone (net 5) (net_name "GND") (layer "B.Cu") (hatch edge 0.508)
+    (connect_pads (clearance 0.508))
+    (min_thickness 0.254) (filled_areas_thickness no)
+    (fill yes (thermal_gap 0.508) (thermal_bridge_width 0.508))
+    (polygon
+      (pts
+        (xy 368.25 167.5)
+        (xy 101.5 167.5)
+        (xy 101.5 78.75)
+        (xy 368.25 78.75)
+      )
+    )
+  )
 )
