File: FrontPanel/FrontPanel.kicad_pcb (KiCad board)
At the start: 2 copper layers, 266.7 x 88.9 mm, 76 parts, among them J1 CPU, J2 Backplane, J3 MPW-Y, U1 74LS38, U2 74LS38, U3 74LS123, U4 NE555P

Commit message: FrontPanel: Provide C4 value
100 nanofarad, looked up by Nakazoto
Parts:
- C4: value C -> 100n
Changed lines of the file:
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@@
       (effects (font (size 1 1) (thickness 0.15)))
     )
-    (fp_text value "C" (at 2.5 2.2 90) (layer "F.Fab")
+    (fp_text value "100n" (at 2.5 2.2 90) (layer "F.Fab")
       (effects (font (size 1 1) (thickness 0.15)))
     )

Commit message: FrontPanel: Improve ground separation
Follow the original idea and fully decouple GND from different connectors.
Parts:
- added C6: 100n, Capacitor_THT:C_Disc_D4.3mm_W1.9mm_P5.00mm, F.Cu at (186.3, 136.4)
- added C7: 100n, Capacitor_THT:C_Disc_D4.3mm_W1.9mm_P5.00mm, F.Cu at (228.7, 136.4)
- added C8: 100n, Capacitor_THT:C_Disc_D4.3mm_W1.9mm_P5.00mm, F.Cu at (260.7, 136.4)
- added C9: 100n, Capacitor_THT:C_Disc_D4.3mm_W1.9mm_P5.00mm, F.Cu at (124.8, 88.6)
- moved R4 23.7 mm to (183.8, 163.0)
Connections:
- net Net-(D1-Pad2) renamed /CL3
- net Net-(D10-Pad2) renamed /A10
- net Net-(D11-Pad2) renamed /A9
- net Net-(D12-Pad2) renamed /A8
- net Net-(D13-Pad2) renamed /A7
- net Net-(D14-Pad2) renamed /A6
- net Net-(D15-Pad2) renamed /A5
- net Net-(D16-Pad2) renamed /A4
- net Net-(D17-Pad2) renamed /A3
- net Net-(D18-Pad2) renamed /A2
- net Net-(D19-Pad2) renamed /A1
- net Net-(D2-Pad2) renamed /CL2
- net Net-(D20-Pad2) renamed /A0
- net Net-(D3-Pad2) renamed /CL1
- net Net-(D4-Pad2) renamed /CL0
- net Net-(D5-Pad2) renamed /A15
- net Net-(D6-Pad2) renamed /A14
- net Net-(D7-Pad2) renamed /A13
- net Net-(D8-Pad2) renamed /A12
- net Net-(D9-Pad2) renamed /A11
- net Net-(J2-Pad11) renamed /~{ResetOut}
- C5 pad 2: GND -> GNDD
- U1 pad 1: GND -> GNDD
- U1 pad 2: GND -> GNDD
- U4 pad 1: GND -> GNDD
Routing:
- net GND: track 499.2 -> 351.3 mm
- net GNDD: track 137.2 -> 240.7 mm
- net Net-(D27-Pad1): track 87.6 -> 98.8 mm
- net Net-(D26-Pad1): track 75.2 -> 83.8 mm
- net +5V: track 526.9 -> 533.4 mm
- net Net-(D24-Pad1): track 58.3 -> 62.7 mm
- net Net-(D25-Pad1): track 76.3 -> 74.7 mm
- net Net-(J1-Pad25): track 63.1 -> 64.5 mm
- added copper zone on B.Cu, net GNDD

Commit message: FrontPanel: Reduce board size
Drop unused space between mounting holes and connectors. This board is fully
compatible with the original while being cheaper due to a smaller area
Parts:
- moved U4 28.7 mm to (106.0, 118.7)
- moved C9 27.7 mm to (112.3, 113.3)
- moved C5 24.6 mm to (119.0, 119.3)
- moved J1 21.2 mm to (195.4, 107.2)
- moved J2 21.2 mm to (287.4, 107.2)
- moved R22 20.6 mm to (121.6, 113.3)
- moved R21 19.8 mm to (116.5, 126.3)
- moved RV1 17.3 mm to (129.0, 113.4)
- moved C1 5.82 mm to (154.3, 120.7)
Routing:
- net +5V: track 533.4 -> 466.5 mm
- net GND: track 351.3 -> 329.6 mm
- net GNDD: track 240.7 -> 219.0 mm
- net Net-(D21-Pad1): track 76.0 -> 54.8 mm
- net /~{ResetFlag}: track 78.8 -> 57.6 mm
- net Net-(D23-Pad1): track 55.4 -> 34.2 mm
- net Net-(D22-Pad1): track 65.7 -> 44.5 mm
- net /A3: track 42.9 -> 21.7 mm
- net /A2: track 53.4 -> 32.3 mm
- net /A1: track 64.0 -> 42.8 mm
- net Net-(J1-Pad7): track 91.9 -> 70.7 mm
- net Net-(D36-Pad1): track 42.5 -> 21.4 mm
- net Net-(J1-Pad4): track 77.0 -> 55.8 mm
- net /A0: track 77.7 -> 56.6 mm
- net Net-(J1-Pad15): track 92.2 -> 73.6 mm
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Other:
- board size 266.7 x 88.9 mm -> 266.7 x 69.8 mm
