File: FrontPanel/FrontPanel.kicad_pcb (KiCad board)
At the start: 2 copper layers, 266.7 x 69.8 mm, 80 parts, among them J1 CPU, J2 Backplane, J3 MPW-Y, U1 74LS38, U2 74LS38, U3 74LS123, U4 NE555P

Commit message: FrontPanel: Erratum E001
Due to unverified assumptions in original schematic, power and ground separation
between connectors, which is actually present on original boards, wasn't done
correctly.
Parts:
- moved RV1 4.02 mm to (133.0, 113.3)
Connections:
- C1 pad 1: +5V -> +5VD
- C6 pad 1: +5V -> +5VD
- C9 pad 1: +5V -> +5VD
- D36 pad 2: +5V -> +5VD
- J1 pad 16: +5V -> +5VD
- J1 pad 18: +5V -> +5VD
- J1 pad 20: +5V -> +5VD
- J1 pad 22: +5V -> +5VD
- J1 pad 24: +5V -> +5VD
- J1 pad 26: +5V -> +5VD
- R12 pad 1: +5V -> +5VD
- R13 pad 1: +5V -> +5VD
- R14 pad 1: +5V -> +5VD
- R15 pad 1: +5V -> +5VD
- R16 pad 1: +5V -> +5VD
- R17 pad 1: +5V -> +5VD
- R18 pad 1: +5V -> +5VD
- R19 pad 1: +5V -> +5VD
- R20 pad 1: +5V -> +5VD
- R22 pad 2: +5V -> +5VD
- R9 pad 1: +5V -> +5VD
- U1 pad 14: +5V -> +5VD
- U4 pad 4: +5V -> +5VD
- U4 pad 8: +5V -> +5VD
Routing:
- net +5V: track 466.5 -> 217.0 mm
- net +5VD: track 0.00 -> 151.3 mm
- net GNDD: track 219.0 -> 194.4 mm
- net Net-(D27-Pad1): track 87.0 -> 74.5 mm
- net Net-(D26-Pad1): track 71.3 -> 59.4 mm
- net Net-(R22-Pad1): track 25.5 -> 29.6 mm
- net Net-(D24-Pad1): track 50.1 -> 46.4 mm
- net Net-(D29-Pad1): track 120.3 -> 122.7 mm
- net Net-(D28-Pad1): track 103.4 -> 105.9 mm
- net Net-(J1-Pad15): track 73.6 -> 71.1 mm
- net Net-(D21-Pad1): track 54.8 -> 57.0 mm
- net Net-(R21-Pad2): track 8.82 -> 10.6 mm
- net Net-(J1-Pad7): track 70.7 -> 71.9 mm
- net Net-(D22-Pad1): track 44.5 -> 45.6 mm
- net Net-(D25-Pad1): track 64.6 -> 63.6 mm
- added copper zone on F.Cu, net +5VD
