File: MUX/MUX.kicad_pcb (KiCad board)
At the start: 4 copper layers, 364 x 203 mm, 139 parts, among them P1 Conn_02x36_Top_Bottom, P2 DB9_Male, P3 DB9_Male, P4 DB9_Male, P5 DB9_Male

Commit message: MUX: Use axial capacitors
Use axial capacitors in order to fully correspond to original board.
Parts:
- C10, C20, C29, C8: footprint Capacitor_THT:CP_Radial_D8.0mm_P3.50mm -> Capacitor_THT:CP_Axial_L25.0mm_D10.0mm_P30.00mm_Horizontal
- moved C10 224.3 mm to (143.9, 216.3), turned to 0 degrees
- moved C8 29.9 mm to (82.7, 34.7), turned to 0 degrees
- moved C20 20.9 mm to (367.2, 61.4), turned to 90 degrees
- moved C29 9.36 mm to (365.8, 188.3), turned to -90 degrees
- moved R13 7.35 mm to (173.5, 208.7), turned to 90 degrees
- moved U_H8 2.16 mm to (168.9, 201.0)
- moved U_K1 1.14 mm to (105.4, 41.8)
Routing:
- net GND: track 3772.2 -> 3813.2 mm
- net +5V: track 3838.8 -> 3802.8 mm
- net Net-(R13-Pad2): track 84.4 -> 97.4 mm
- net Sys.~{A_{0}}: track 41.6 -> 51.8 mm
- net Sys.~{A_{1}}: track 49.9 -> 55.0 mm
- net +12V: track 562.0 -> 566.3 mm
- net Sys.~{INTACK}: track 54.1 -> 58.0 mm
- net Sys.INT_IN: track 46.7 -> 50.6 mm
- net Sys.~{A_{7}}: track 53.8 -> 50.3 mm
- net Sys.~{A_{8}}: track 62.5 -> 59.0 mm
- net Sys.~{A_{4}}: track 60.5 -> 56.9 mm
- net /~{Reset}: track 431.9 -> 435.4 mm
- net Sys.~{A_{5}}: track 69.3 -> 66.0 mm
- net Net-(U_H7-Pad9): track 117.0 -> 114.0 mm
- net Sys.~{A_{2}}: track 59.0 -> 61.9 mm
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