File: DebugInterface/DebugInterface.kicad_sch (KiCad schematic)
At the start: 37 parts, among them J1 IDC-50M, J10 Barrel_Jack_MountingPin, J11 ISP, J2 IDC-50M, J3 IDC-50M, J4 IDC-50M, J5 IDC-50M, J6 IDC-50M, J7 IDC-50M, J8 IDC-50M, J9 USB_B, U1 8255, U10 PIC18F2550-ISO, U2 8255, U3 8255, U4 8255, U5 8255, U6 8255, U7 8255, U8 8255, U9 74LS138, Y1 20MHz

Commit message: DebugInterface: Redone with PIC18
Better I/O ports and normal USB.
Parts:
- added C9: 100nF, Capacitor_THT:C_Disc_D4.3mm_W1.9mm_P5.00mm, symbol Device:C
- C1: renamed from C5; footprint (none) -> Capacitor_THT:C_Disc_D4.3mm_W1.9mm_P5.00mm
- C10: renamed from C1; footprint (none) -> Capacitor_THT:C_Disc_D4.3mm_W1.9mm_P5.00mm
- C11: renamed from C2; footprint (none) -> Capacitor_THT:C_Disc_D4.3mm_W1.9mm_P5.00mm
- C12: renamed from C3; footprint (none) -> Capacitor_THT:C_Disc_D4.3mm_W1.9mm_P5.00mm
- C13: renamed from C4; footprint (none) -> Capacitor_THT:C_Disc_D4.3mm_W1.9mm_P5.00mm
- C14: renamed from C13; footprint (none) -> Capacitor_THT:CP_Radial_D8.0mm_P3.80mm
- C2: renamed from C6; footprint (none) -> Capacitor_THT:C_Disc_D4.3mm_W1.9mm_P5.00mm
- C3: renamed from C7; footprint (none) -> Capacitor_THT:C_Disc_D4.3mm_W1.9mm_P5.00mm
- C4: renamed from C8; footprint (none) -> Capacitor_THT:C_Disc_D4.3mm_W1.9mm_P5.00mm
- C5: renamed from C9; footprint (none) -> Capacitor_THT:C_Disc_D4.3mm_W1.9mm_P5.00mm
- C6: renamed from C10; footprint (none) -> Capacitor_THT:C_Disc_D4.3mm_W1.9mm_P5.00mm
- C7: renamed from C11; footprint (none) -> Capacitor_THT:C_Disc_D4.3mm_W1.9mm_P5.00mm
- C8: renamed from C12; footprint (none) -> Capacitor_THT:C_Disc_D4.3mm_W1.9mm_P5.00mm
- J9: footprint (none) -> Connector_USB:USB_B_OST_USB-B1HSxx_Horizontal
- R1, R2: footprint (none) -> Resistor_THT:R_Axial_DIN0207_L6.3mm_D2.5mm_P10.16mm_Horizontal
- U9: footprint (none) -> DIP-16_W7.62mm
- Y1: footprint (none) -> Crystal:Crystal_HC49-U_Vertical
Connections:
- net GND: now also C9.2
- net RST: now also U10.11 (T1OSO/T13CKI/RC0); no longer U10.13 (CCP1/RC2)
- net VCC: now also C9.1
- net ~{RD}: now also U10.13 (CCP1/RC2); no longer U10.11 (T1OSO/T13CKI/RC0)
Other:
- moved on the sheet: C14

Commit message: DebugInterface: Fix ISP connector
Proper pin assignment
Connections:
- net D5: now also J11.6 (Pin_6); no longer J11.4 (Pin_4)
- net D7: now also J11.4 (Pin_4); no longer J11.6 (Pin_6)
Changed lines of the file:
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@@
-    (effects (font (size 1.27 1.27)) (justify left bottom))
-  )
-  (label "D7" (at 387.35 227.33 0) (fields_autoplaced)
     (effects (font (size 1.27 1.27)) (justify left bottom))
   )
@@
     (effects (font (size 1.27 1.27)) (justify left bottom))
   )
-  (label "D5" (at 387.35 222.25 0) (fields_autoplaced)
-    (effects (font (size 1.27 1.27)) (justify left bottom))
-  )
   (label "RST" (at 223.52 158.75 0) (fields_autoplaced)
     (effects (font (size 1.27 1.27)) (justify left bottom))
@@
     (effects (font (size 1.27 1.27)) (justify left bottom))
   )
+  (label "D7" (at 387.35 222.25 0) (fields_autoplaced)
+    (effects (font (size 1.27 1.27)) (justify left bottom))
+  )
   (label "RST" (at 146.05 158.75 0) (fields_autoplaced)
     (effects (font (size 1.27 1.27)) (justify left bottom))
@@
     (effects (font (size 1.27 1.27)) (justify left bottom))
   )
+  (label "D5" (at 387.35 227.33 0) (fields_autoplaced)
+    (effects (font (size 1.27 1.27)) (justify left bottom))
+  )

Commit message: DebugInterface: Second version
Each port has got own connector for ease of separation and making cables.
Ports are rearranged in address space to enable longer sequential
reads/writes
Parts:
- removed J1, J2, J3, J4, J5, J6, J7, J8: IDC-50M, Connector_IDC:IDC-Header_2x25_P2.54mm_Vertical, symbol Connector_Generic:Conn_02x25_Odd_Even
- added J1, J10, J11, J12, J13, J14, J15, J16, J17, J18, J19, J2, J20, J21, J22, J23, J24, J3, J4, J5, J6, J7, J8, J9: IDC-16M, Connector_IDC:IDC-Header_2x08_P2.54mm_Vertical, symbol Connector_Generic:Conn_02x08_Odd_Even
- renumbered J9 to J25, J11 to J26, J10 to J27, U3 to U2, U5 to U3, U7 to U4, U2 to U5, U4 to U6, U6 to U7
Connections:
- net A0: now also U9.1 (A0); no longer U1.9 (A0), U2.9 (A0), U3.9 (A0), U4.9 (A0), U5.9 (A0), U6.9 (A0), U7.9 (A0), U8.9 (A0)
- net A1: now also U9.2 (A1); no longer U1.8 (A1), U2.8 (A1), U3.8 (A1), U4.8 (A1), U5.8 (A1), U6.8 (A1), U7.8 (A1), U8.8 (A1)
- net A2: now also U9.3 (A2); no longer U9.1 (A0)
- net A3: now also U1.9 (A0), U2.9 (A0), U3.9 (A0), U4.9 (A0), U5.9 (A0), U6.9 (A0), U7.9 (A0), U8.9 (A0); no longer U9.2 (A1)
- net A4: now also U1.8 (A1), U2.8 (A1), U3.8 (A1), U4.8 (A1), U5.8 (A1), U6.8 (A1), U7.8 (A1), U8.8 (A1); no longer U9.3 (A2)
- net GND: now also J1.1 (Pin_1), J1.11 (Pin_11), J1.13 (Pin_13), J1.15 (Pin_15), J1.3 (Pin_3), J1.5 (Pin_5), J1.7 (Pin_7), J1.9 (Pin_9), J10.1 (Pin_1), J10.11 (Pin_11), J10.13 (Pin_13), J10.15 (Pin_15), J10.3 (Pin_3), J10.5 (Pin_5), J10.7 (Pin_7), J10.9 (Pin_9), J11.1 (Pin_1), J11.11 (Pin_11), J11.13 (Pin_13), J11.15 (Pin_15), J11.3 (Pin_3), J11.5 (Pin_5), J11.7 (Pin_7), J11.9 (Pin_9), J12.1 (Pin_1), J12.11 (Pin_11), J12.13 (Pin_13), J12.15 (Pin_15), J12.3 (Pin_3), J12.5 (Pin_5), J12.7 (Pin_7), J12.9 (Pin_9), J13.1 (Pin_1), J13.11 (Pin_11), J13.13 (Pin_13), J13.15 (Pin_15), J13.3 (Pin_3), J13.5 (Pin_5), J13.7 (Pin_7), J13.9 (Pin_9), J14.1 (Pin_1), J14.11 (Pin_11), J14.13 (Pin_13), J14.15 (Pin_15), J14.3 (Pin_3), J14.5 (Pin_5), J14.7 (Pin_7), J14.9 (Pin_9), J15.1 (Pin_1), J15.11 (Pin_11), J15.13 (Pin_13), J15.15 (Pin_15), J15.3 (Pin_3), J15.5 (Pin_5), J15.7 (Pin_7), J15.9 (Pin_9), J16.1 (Pin_1), J16.11 (Pin_11), J16.13 (Pin_13), J16.15 (Pin_15), J16.3 (Pin_3), J16.5 (Pin_5), J16.7 (Pin_7), J16.9 (Pin_9), J17.1 (Pin_1), J17.11 (Pin_11), J17.13 (Pin_13), J17.15 (Pin_15), J17.3 (Pin_3), J17.5 (Pin_5), J17.7 (Pin_7), J17.9 (Pin_9), J18.1 (Pin_1), J18.11 (Pin_11), J18.13 (Pin_13), J18.15 (Pin_15), J18.3 (Pin_3), J18.5 (Pin_5), J18.7 (Pin_7), J18.9 (Pin_9), J19.1 (Pin_1), J19.11 (Pin_11), J19.13 (Pin_13), J19.15 (Pin_15), J19.3 (Pin_3), J19.5 (Pin_5), J19.7 (Pin_7), J19.9 (Pin_9), J2.1 (Pin_1), J2.11 (Pin_11), J2.13 (Pin_13), J2.15 (Pin_15), J2.3 (Pin_3), J2.5 (Pin_5), J2.7 (Pin_7), J2.9 (Pin_9), J20.1 (Pin_1), J20.11 (Pin_11), J20.13 (Pin_13), J20.15 (Pin_15), J20.3 (Pin_3), J20.5 (Pin_5), J20.7 (Pin_7), J20.9 (Pin_9), J21.1 (Pin_1), J21.11 (Pin_11), J21.13 (Pin_13), J21.15 (Pin_15), J21.3 (Pin_3), J21.5 (Pin_5), J21.7 (Pin_7), J21.9 (Pin_9), J22.1 (Pin_1), J22.11 (Pin_11), J22.13 (Pin_13), J22.15 (Pin_15), J22.3 (Pin_3), J22.5 (Pin_5), J22.7 (Pin_7), J22.9 (Pin_9), J23.1 (Pin_1), J23.11 (Pin_11), J23.13 (Pin_13), J23.15 (Pin_15), J23.3 (Pin_3), J23.5 (Pin_5), J23.7 (Pin_7), J23.9 (Pin_9), J24.1 (Pin_1), J24.11 (Pin_11), J24.13 (Pin_13), J24.15 (Pin_15), J24.3 (Pin_3), J24.5 (Pin_5), J24.7 (Pin_7), J24.9 (Pin_9), J3.1 (Pin_1), J3.11 (Pin_11), J3.13 (Pin_13), J3.15 (Pin_15), J3.3 (Pin_3), J3.5 (Pin_5), J3.7 (Pin_7), J3.9 (Pin_9), J4.1 (Pin_1), J4.11 (Pin_11), J4.13 (Pin_13), J4.15 (Pin_15), J4.3 (Pin_3), J4.5 (Pin_5), J4.7 (Pin_7), J4.9 (Pin_9), J5.1 (Pin_1), J5.11 (Pin_11), J5.13 (Pin_13), J5.15 (Pin_15), J5.3 (Pin_3), J5.5 (Pin_5), J5.7 (Pin_7), J5.9 (Pin_9), J6.1 (Pin_1), J6.11 (Pin_11), J6.13 (Pin_13), J6.15 (Pin_15), J6.3 (Pin_3), J6.5 (Pin_5), J6.7 (Pin_7), J6.9 (Pin_9), J7.1 (Pin_1), J7.11 (Pin_11), J7.13 (Pin_13), J7.15 (Pin_15), J7.3 (Pin_3), J7.5 (Pin_5), J7.7 (Pin_7), J7.9 (Pin_9), J8.1 (Pin_1), J8.11 (Pin_11), J8.13 (Pin_13), J8.15 (Pin_15), J8.3 (Pin_3), J8.5 (Pin_5), J8.7 (Pin_7), J8.9 (Pin_9), J9.1 (Pin_1), J9.11 (Pin_11), J9.13 (Pin_13), J9.15 (Pin_15), J9.3 (Pin_3), J9.5 (Pin_5), J9.7 (Pin_7), J9.9 (Pin_9)
- net ~{CS1}: now also U2.6 (~{CS}); no longer U5.6 (~{CS})
- net ~{CS2}: now also U3.6 (~{CS}); no longer U2.6 (~{CS})
- net ~{CS3}: now also U4.6 (~{CS}); no longer U6.6 (~{CS})
- net ~{CS4}: now also U5.6 (~{CS}); no longer U3.6 (~{CS})
- net ~{CS5}: now also U6.6 (~{CS}); no longer U7.6 (~{CS})
- net ~{CS6}: now also U7.6 (~{CS}); no longer U4.6 (~{CS})
- net at U2.1 (PA3): now also J4.8 (Pin_8)
- net at U2.10 (PC7): now also J6.16 (Pin_16)
- net at U2.11 (PC6): now also J6.14 (Pin_14)
- net at U2.12 (PC5): now also J6.12 (Pin_12)
- net at U2.13 (PC4): now also J6.10 (Pin_10)
- net at U2.14 (PC0): now also J6.2 (Pin_2)
- net at U2.15 (PC1): now also J6.4 (Pin_4)
- net at U2.16 (PC2): now also J6.6 (Pin_6)
- net at U2.17 (PC3): now also J6.8 (Pin_8)
- net at U2.18 (PB0): now also J5.2 (Pin_2)
- net at U2.19 (PB1): now also J5.4 (Pin_4)
- net at U2.2 (PA2): now also J4.6 (Pin_6)
- net at U2.20 (PB2): now also J5.6 (Pin_6)
- net at U2.21 (PB3): now also J5.8 (Pin_8)
- net at U2.22 (PB4): now also J5.10 (Pin_10)
- net at U2.23 (PB5): now also J5.12 (Pin_12)
- net at U2.24 (PB6): now also J5.14 (Pin_14)
- net at U2.25 (PB7): now also J5.16 (Pin_16)
- net at U2.3 (PA1): now also J4.4 (Pin_4)
- net at U2.37 (PA7): now also J4.16 (Pin_16)
- net at U2.38 (PA6): now also J4.14 (Pin_14)
- net at U2.39 (PA5): now also J4.12 (Pin_12)
- net at U2.4 (PA0): now also J4.2 (Pin_2)
- net at U2.40 (PA4): now also J4.10 (Pin_10)
- net at U4.40 (PA4): now also J10.10 (Pin_10)
- net at U4.39 (PA5): now also J10.12 (Pin_12)
- net at U4.38 (PA6): now also J10.14 (Pin_14)
- net at U4.37 (PA7): now also J10.16 (Pin_16)
- net at U4.18 (PB0): now also J11.2 (Pin_2)
- net at U4.4 (PA0): now also J10.2 (Pin_2)
- net at U4.19 (PB1): now also J11.4 (Pin_4)
- net at U4.20 (PB2): now also J11.6 (Pin_6)
- net at U4.21 (PB3): now also J11.8 (Pin_8)
- net at U4.22 (PB4): now also J11.10 (Pin_10)
- net at U4.23 (PB5): now also J11.12 (Pin_12)
- net at U4.24 (PB6): now also J11.14 (Pin_14)
- net at U4.25 (PB7): now also J11.16 (Pin_16)
- net at U4.14 (PC0): now also J12.2 (Pin_2)
- net at U4.15 (PC1): now also J12.4 (Pin_4)
- net at U4.16 (PC2): now also J12.6 (Pin_6)
- net at U4.3 (PA1): now also J10.4 (Pin_4)
- net at U4.17 (PC3): now also J12.8 (Pin_8)
- net at U4.13 (PC4): now also J12.10 (Pin_10)
- net at U4.12 (PC5): now also J12.12 (Pin_12)
- net at U4.11 (PC6): now also J12.14 (Pin_14)
- net at U4.10 (PC7): now also J12.16 (Pin_16)
- net at U4.2 (PA2): now also J10.6 (Pin_6)
- net at U4.1 (PA3): now also J10.8 (Pin_8)
- net at U1.40 (PA4): now also J1.10 (Pin_10)
- net at U1.39 (PA5): now also J1.12 (Pin_12)
- net at U1.38 (PA6): now also J1.14 (Pin_14)
- net at U1.37 (PA7): now also J1.16 (Pin_16)
- net at U1.18 (PB0): now also J2.2 (Pin_2)
- net at U1.4 (PA0): now also J1.2 (Pin_2)
- net at U1.19 (PB1): now also J2.4 (Pin_4)
- net at U1.20 (PB2): now also J2.6 (Pin_6)
- net at U1.21 (PB3): now also J2.8 (Pin_8)
- net at U1.22 (PB4): now also J2.10 (Pin_10)
- net at U1.23 (PB5): now also J2.12 (Pin_12)
- net at U1.24 (PB6): now also J2.14 (Pin_14)
- net at U1.25 (PB7): now also J2.16 (Pin_16)
- net at U1.14 (PC0): now also J3.2 (Pin_2)
- net at U1.15 (PC1): now also J3.4 (Pin_4)
- net at U1.16 (PC2): now also J3.6 (Pin_6)
- net at U1.3 (PA1): now also J1.4 (Pin_4)
- net at U1.17 (PC3): now also J3.8 (Pin_8)
- net at U1.13 (PC4): now also J3.10 (Pin_10)
- net at U1.12 (PC5): now also J3.12 (Pin_12)
- net at U1.11 (PC6): now also J3.14 (Pin_14)
- net at U1.10 (PC7): now also J3.16 (Pin_16)
- net at U1.2 (PA2): now also J1.6 (Pin_6)
- net at U1.1 (PA3): now also J1.8 (Pin_8)
- net at U7.1 (PA3): now also J19.8 (Pin_8)
- net at U7.10 (PC7): now also J21.16 (Pin_16)
- net at U7.11 (PC6): now also J21.14 (Pin_14)
- net at U7.12 (PC5): now also J21.12 (Pin_12)
- net at U7.13 (PC4): now also J21.10 (Pin_10)
- net at U7.14 (PC0): now also J21.2 (Pin_2)
- net at U7.15 (PC1): now also J21.4 (Pin_4)
- net at U7.16 (PC2): now also J21.6 (Pin_6)
- net at U7.17 (PC3): now also J21.8 (Pin_8)
- net at U7.18 (PB0): now also J20.2 (Pin_2)
- net at U7.19 (PB1): now also J20.4 (Pin_4)
- net at U7.2 (PA2): now also J19.6 (Pin_6)
- net at U7.20 (PB2): now also J20.6 (Pin_6)
- net at U7.21 (PB3): now also J20.8 (Pin_8)
- net at U7.22 (PB4): now also J20.10 (Pin_10)
- net at U7.23 (PB5): now also J20.12 (Pin_12)
- net at U7.24 (PB6): now also J20.14 (Pin_14)
- net at U7.25 (PB7): now also J20.16 (Pin_16)
- net at U7.3 (PA1): now also J19.4 (Pin_4)
- net at U7.37 (PA7): now also J19.16 (Pin_16)
- net at U7.38 (PA6): now also J19.14 (Pin_14)
- net at U7.39 (PA5): now also J19.12 (Pin_12)
- net at U7.4 (PA0): now also J19.2 (Pin_2)
- net at U7.40 (PA4): now also J19.10 (Pin_10)
- net at U5.40 (PA4): now also J13.10 (Pin_10)
- net at U5.39 (PA5): now also J13.12 (Pin_12)
- net at U5.38 (PA6): now also J13.14 (Pin_14)
- net at U5.37 (PA7): now also J13.16 (Pin_16)
- net at U5.18 (PB0): now also J14.2 (Pin_2)
- net at U5.4 (PA0): now also J13.2 (Pin_2)
- net at U5.19 (PB1): now also J14.4 (Pin_4)
- net at U5.20 (PB2): now also J14.6 (Pin_6)
- net at U5.21 (PB3): now also J14.8 (Pin_8)
- net at U5.22 (PB4): now also J14.10 (Pin_10)
- net at U5.23 (PB5): now also J14.12 (Pin_12)
- net at U5.24 (PB6): now also J14.14 (Pin_14)
- net at U5.25 (PB7): now also J14.16 (Pin_16)
- net at U5.14 (PC0): now also J15.2 (Pin_2)
- net at U5.15 (PC1): now also J15.4 (Pin_4)
- net at U5.16 (PC2): now also J15.6 (Pin_6)
- net at U5.3 (PA1): now also J13.4 (Pin_4)
- net at U5.17 (PC3): now also J15.8 (Pin_8)
- net at U5.13 (PC4): now also J15.10 (Pin_10)
- net at U5.12 (PC5): now also J15.12 (Pin_12)
- net at U5.11 (PC6): now also J15.14 (Pin_14)
- net at U5.10 (PC7): now also J15.16 (Pin_16)
- net at U5.2 (PA2): now also J13.6 (Pin_6)
- net at U5.1 (PA3): now also J13.8 (Pin_8)
- net at U8.1 (PA3): now also J22.8 (Pin_8)
- net at U8.10 (PC7): now also J24.16 (Pin_16)
- net at U8.11 (PC6): now also J24.14 (Pin_14)
- net at U8.12 (PC5): now also J24.12 (Pin_12)
- net at U8.13 (PC4): now also J24.10 (Pin_10)
- net at U8.14 (PC0): now also J24.2 (Pin_2)
- net at U8.15 (PC1): now also J24.4 (Pin_4)
- net at U8.16 (PC2): now also J24.6 (Pin_6)
- net at U8.17 (PC3): now also J24.8 (Pin_8)
- net at U8.18 (PB0): now also J23.2 (Pin_2)
- net at U8.19 (PB1): now also J23.4 (Pin_4)
- net at U8.2 (PA2): now also J22.6 (Pin_6)
- net at U8.20 (PB2): now also J23.6 (Pin_6)
- net at U8.21 (PB3): now also J23.8 (Pin_8)
- net at U8.22 (PB4): now also J23.10 (Pin_10)
- net at U8.23 (PB5): now also J23.12 (Pin_12)
- net at U8.24 (PB6): now also J23.14 (Pin_14)
- net at U8.25 (PB7): now also J23.16 (Pin_16)
- net at U8.3 (PA1): now also J22.4 (Pin_4)
- net at U8.37 (PA7): now also J22.16 (Pin_16)
- net at U8.38 (PA6): now also J22.14 (Pin_14)
- net at U8.39 (PA5): now also J22.12 (Pin_12)
- net at U8.4 (PA0): now also J22.2 (Pin_2)
- net at U8.40 (PA4): now also J22.10 (Pin_10)
- net at U6.40 (PA4): now also J16.10 (Pin_10)
- net at U6.39 (PA5): now also J16.12 (Pin_12)
- net at U6.38 (PA6): now also J16.14 (Pin_14)
- net at U6.37 (PA7): now also J16.16 (Pin_16)
- net at U6.18 (PB0): now also J17.2 (Pin_2)
- net at U6.4 (PA0): now also J16.2 (Pin_2)
- net at U6.19 (PB1): now also J17.4 (Pin_4)
- net at U6.20 (PB2): now also J17.6 (Pin_6)
- net at U6.21 (PB3): now also J17.8 (Pin_8)
- net at U6.22 (PB4): now also J17.10 (Pin_10)
- net at U6.23 (PB5): now also J17.12 (Pin_12)
- net at U6.24 (PB6): now also J17.14 (Pin_14)
- net at U6.25 (PB7): now also J17.16 (Pin_16)
- net at U6.14 (PC0): now also J18.2 (Pin_2)
- net at U6.15 (PC1): now also J18.4 (Pin_4)
- net at U6.16 (PC2): now also J18.6 (Pin_6)
- net at U6.3 (PA1): now also J16.4 (Pin_4)
- net at U6.17 (PC3): now also J18.8 (Pin_8)
- net at U6.13 (PC4): now also J18.10 (Pin_10)
- net at U6.12 (PC5): now also J18.12 (Pin_12)
- net at U6.11 (PC6): now also J18.14 (Pin_14)
- net at U6.10 (PC7): now also J18.16 (Pin_16)
- net at U6.2 (PA2): now also J16.6 (Pin_6)
- net at U6.1 (PA3): now also J16.8 (Pin_8)
- net at U3.40 (PA4): now also J7.10 (Pin_10)
- net at U3.39 (PA5): now also J7.12 (Pin_12)
- net at U3.38 (PA6): now also J7.14 (Pin_14)
- net at U3.37 (PA7): now also J7.16 (Pin_16)
- net at U3.18 (PB0): now also J8.2 (Pin_2)
- net at U3.4 (PA0): now also J7.2 (Pin_2)
- net at U3.19 (PB1): now also J8.4 (Pin_4)
- net at U3.20 (PB2): now also J8.6 (Pin_6)
- net at U3.21 (PB3): now also J8.8 (Pin_8)
- net at U3.22 (PB4): now also J8.10 (Pin_10)
- net at U3.23 (PB5): now also J8.12 (Pin_12)
- net at U3.24 (PB6): now also J8.14 (Pin_14)
- net at U3.25 (PB7): now also J8.16 (Pin_16)
- net at U3.14 (PC0): now also J9.2 (Pin_2)
- net at U3.15 (PC1): now also J9.4 (Pin_4)
- net at U3.16 (PC2): now also J9.6 (Pin_6)
- net at U3.3 (PA1): now also J7.4 (Pin_4)
- net at U3.17 (PC3): now also J9.8 (Pin_8)
- net at U3.13 (PC4): now also J9.10 (Pin_10)
- net at U3.12 (PC5): now also J9.12 (Pin_12)
- net at U3.11 (PC6): now also J9.14 (Pin_14)
- net at U3.10 (PC7): now also J9.16 (Pin_16)
- net at U3.2 (PA2): now also J7.6 (Pin_6)
- net at U3.1 (PA3): now also J7.8 (Pin_8)
- no-connect marks 9 -> 2

Commit message: DebugInterface: Add some LEDs
Some indicator LEDs: power, reset, activity.
Parts:
- added D1, D2, D3, D4: LED, LED_THT:LED_D3.0mm, symbol Device:LED
- added R3, R4, R5, R6: 1K, Resistor_THT:R_Axial_DIN0207_L6.3mm_D2.5mm_P10.16mm_Horizontal, symbol Device:R
Connections:
- net GND: now also D1.1 (K), D2.1 (K), D3.1 (K), D4.1 (K)
- net RST: now also U9.4 (E1), R4.1
- net VCC: now also R3.1
- net at C13.1, J25.1 (VBUS), J26.2 (Pin_2)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: now also R5.1
- net at U10.17 (TX/CK/RC6): now also R6.1
- net ~{AEN}: no longer names the net of U10.7 (RA5/AN4/~{SS}/HLVDIN/C2OUT)
- net ~{AEN}: no longer U9.4 (E1)
- new net: D2.2 (A), R6.2
- new net: D1.2 (A), R5.2
- new net: D3.2 (A), R3.2
- new net: D4.2 (A), R4.2
Other:
- moved on the sheet: R1, U9

Commit message: DebugInterface: Final preps
A bit of layout optimization, LED designations on silkscreen
Parts:
- D1: value LED -> VUSB
- D2: value LED -> ACT
- D3: value LED -> VCC
- D4: value LED -> RST
Changed lines of the file:
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@@
 			)
 		)
-		(property "Value" "LED"
+		(property "Value" "ACT"
 			(at 396.494 230.124 90)
 			(effects
@@
 			)
 		)
-		(property "Value" "LED"
+		(property "Value" "VUSB"
 			(at 403.098 230.124 90)
 			(effects
@@
 		(on_board yes)
 		(dnp no)
-		(fields_autoplaced yes)
 		(property "Reference" "D3"
 			(at 246.38 272.0974 90)
@@
 			)
 		)
-		(property "Value" "LED"
+		(property "Value" "VCC"
 			(at 246.38 274.6374 90)
 			(effects
@@
 			)
 		)
-		(property "Value" "LED"
+		(property "Value" "RST"
 			(at 256.54 274.6374 90)
 			(effects
