File: DiagBoard/Diag.kicad_sch (KiCad schematic)
At the start: 80 parts, among them J1 B1, P1 Conn_02x36_Top_Bottom, SW1 SW_DIP_x07, SW2 SW_Push, SW3 SW_DIP_x04

Commit message: DiagBoard: Revert to TIL311
It turns out that a discrete indicator with two DPs is no less unobtanium.
Actually, TIL311 are widely available, albeit expensive. Well, rebuilding a
minicomputer is no cheap feat
Parts:
- removed AFF1, AFF2: LTS-6960HR, Display_7Segment:7SegmentLED_LTS6760_LTS6780, symbol Display_Character:LTS-6960HR
- removed R10, R11, R12, R13, R14, R15, R16, R17, R18, R19, R20, R21, R22, R9: 220, Resistor_THT:R_Axial_DIN0204_L3.6mm_D1.6mm_P5.08mm_Horizontal, symbol Device:R
- removed U_X2, U_X3: N8223B, Package_DIP:DIP-16_W7.62mm, symbol 74xx:74LS259
- removed U_X2: 74LS574, Package_DIP:DIP-20_W7.62mm, symbol 74xx:74LS574
- added DIS1, DIS2: TIL311, Package_DIP:DIP-14_W7.62mm, symbol led-displays-obsolete:TIL311
- added RN2: 4.7K, Resistor_THT:R_Array_SIP10, symbol Device:R_Network09
- RN1: footprint Resistor_THT:R_Array_SIP9 -> Resistor_THT:R_Array_SIP10; symbol Device:R_Network08 -> Device:R_Network09
- renumbered R4 to R1, R3 to R2, R1 to R3, R2 to R4
Connections:
- net +5V: now also DIS1.1 (Vcc_LED), DIS1.14 (Vcc_logic), DIS2.1 (Vcc_LED), DIS2.14 (Vcc_logic), RN2.1 (common)
- net BLNK: now also DIS1.8 (Blanking_Input), DIS2.8 (Blanking_Input)
- net D0_O: now also DIS2.3 (A)
- net D1_O: now also DIS2.2 (B)
- net D2_O: now also DIS2.13 (C)
- net D3_O: now also DIS2.12 (D)
- net D4_O: now also DIS1.3 (A)
- net D5_O: now also DIS1.2 (B)
- net D6_O: now also DIS1.13 (C)
- net D7_O: now also DIS1.12 (D)
- net GND: now also SW2.1, DIS1.7 (GND), DIS2.7 (GND)
- net DIAG_MEM: now reaches U_A1.1, U_A1.12, U_A1.13, U_A1.2, U_C3.6 (Oa=b), U_D1.5, U_J6.1
- net at SW1.10, U_K7.14 (D5): now also RN2.8 (R7)
- net at SW1.11, U_K7.13 (D4): now also RN2.7 (R6)
- net at SW1.12, U_K7.3 (D0): now also RN2.6 (R5)
- net at SW1.13, U_K7.4 (D1): now also RN2.5 (R4)
- net at SW1.14, U_K7.7 (D2): now also RN2.4 (R3)
- net at SW1.8, U_K7.18 (D7): now also RN2.10 (R9)
- net at SW1.9, U_K7.17 (D6): now also RN2.9 (R8)
- net at R1.1: now also DIS1.10 (Right_Decimal)
- net at R3.1: now also DIS2.10 (Right_Decimal)
- net at C1.1, D1.2 (A), SW2.2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: now also RN2.3 (R2)
- net at R2.1: now also DIS1.4 (Left_Decimal)
- net at R4.1: now also DIS2.4 (Left_Decimal)
- net STRB renamed ~{STRB}
- net ~{STRB}: now also DIS1.5 (/Latch_Strobe_Input), DIS2.5 (/Latch_Strobe_Input)
- no-connect marks 59 -> 58
Other:
- note added: "Memory base address selector"
- note added: "Memory data gate"
- note removed: "TODO: Resistor network missing ?"
- moved on the sheet: C1, C2, C3, D1, J1, P1, R1, R2, R3, R4, R5, R6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

Commit message: Fix U_C8 type
It's 74LS08
Parts:
- U_C8: value 74LS38 -> 74LS08; symbol 74xx:74LS38 -> 74xx:74LS08
Changed lines of the file:
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@@
 	)
 	(symbol
-		(lib_id "74xx:74LS38")
+		(lib_id "74xx:74LS08")
 		(at 725.17 132.08 0)
 		(unit 1)
@@
 			)
 		)
-		(property "Value" "74LS38"
+		(property "Value" "74LS08"
 			(at 725.1617 125.73 0)
 			(effects
@@
 			)
 		)
-		(property "Datasheet" "http://www.ti.com/lit/gpn/sn74LS38"
+		(property "Datasheet" "http://www.ti.com/lit/gpn/sn74LS08"
 			(at 725.17 132.08 0)
 			(effects
@@
 			)
 		)
-		(property "Description" "Quad Buffer 2-input NAND Open collector"
+		(property "Description" "Quad And2"
 			(at 725.17 132.08 0)
 			(effects
@@
 	)
 	(symbol
-		(lib_id "74xx:74LS38")
+		(lib_id "74xx:74LS08")
 		(at 725.17 147.32 0)
 		(unit 2)
@@
 			)
 		)
-		(property "Value" "74LS38"
+		(property "Value" "74LS08"
 			(at 725.1617 140.97 0)
 			(effects
@@
 			)
 		)
-		(property "Datasheet" "http://www.ti.com/lit/gpn/sn74LS38"
+		(property "Datasheet" "http://www.ti.com/lit/gpn/sn74LS08"
 			(at 725.17 147.32 0)
 			(effects
@@
 			)
 		)
-		(property "Description" "Quad Buffer 2-input NAND Open collector"
+		(property "Description" "Quad And2"
 			(at 725.17 147.32 0)
 			(effects
