File: DiagBoard/DiagBoard.kicad_pcb (KiCad board)
At the start: 4 copper layers, 364 x 203 mm, 67 parts, among them J1 B1, P1 Conn_02x36_Top_Bottom, SW1 SW_DIP_x07, SW2 SW_Push_DPDT, SW3 SW_DIP_x04

Commit message: DiagBoard: Complete reconstruction
Complete with extra functionality and connectors for experiments
Parts:
- added C10: 100n, Capacitor_THT:C_Disc_D4.3mm_W1.9mm_P5.00mm, F.Cu at (156.0, 48.0)
- added C11: 100n, Capacitor_THT:C_Disc_D4.3mm_W1.9mm_P5.00mm, F.Cu at (155.0, 70.0)
- added C12: 100n, Capacitor_THT:C_Disc_D4.3mm_W1.9mm_P5.00mm, F.Cu at (155.3, 91.9)
- added C13: 100n, Capacitor_THT:C_Disc_D4.3mm_W1.9mm_P5.00mm, F.Cu at (155.3, 113.9)
- added C14: 100n, Capacitor_THT:C_Disc_D4.3mm_W1.9mm_P5.00mm, F.Cu at (155.3, 135.9)
- added C15: 100n, Capacitor_THT:C_Disc_D4.3mm_W1.9mm_P5.00mm, F.Cu at (155.3, 157.9)
- added C16: 100n, Capacitor_THT:C_Disc_D4.3mm_W1.9mm_P5.00mm, F.Cu at (153.5, 173.2)
- added C17: 100n, Capacitor_THT:C_Disc_D4.3mm_W1.9mm_P5.00mm, F.Cu at (155.3, 204.2)
- added C18: 100n, Capacitor_THT:C_Disc_D4.3mm_W1.9mm_P5.00mm, F.Cu at (229.0, 110.9)
- added C19: 100n, Capacitor_THT:C_Disc_D4.3mm_W1.9mm_P5.00mm, F.Cu at (256.4, 49.4)
- added C20: 100n, Capacitor_THT:C_Disc_D4.3mm_W1.9mm_P5.00mm, F.Cu at (256.4, 73.1)
- added C21: 100n, Capacitor_THT:C_Disc_D4.3mm_W1.9mm_P5.00mm, F.Cu at (256.4, 91.2)
- added C22: 100n, Capacitor_THT:C_Disc_D4.3mm_W1.9mm_P5.00mm, F.Cu at (256.4, 130.0)
- added C23: 100n, Capacitor_THT:C_Disc_D4.3mm_W1.9mm_P5.00mm, F.Cu at (256.4, 178.7)
- added C24: 100n, Capacitor_THT:C_Disc_D4.3mm_W1.9mm_P5.00mm, F.Cu at (256.4, 204.2)
- added C25: 100n, Capacitor_THT:C_Disc_D4.3mm_W1.9mm_P5.00mm, F.Cu at (284.7, 110.9)
- added C26: 100n, Capacitor_THT:C_Disc_D4.3mm_W1.9mm_P5.00mm, F.Cu at (314.2, 49.4)
- added C27: 100n, Capacitor_THT:C_Disc_D4.3mm_W1.9mm_P5.00mm, F.Cu at (332.4, 72.2)
- added C28: 100n, Capacitor_THT:C_Rect_L9.0mm_W2.5mm_P7.50mm_MKT, F.Cu at (332.4, 92.3)
- added C29: 100n, Capacitor_THT:C_Disc_D4.3mm_W1.9mm_P5.00mm, F.Cu at (332.2, 110.9)
- added C30: 100n, Capacitor_THT:C_Disc_D4.3mm_W1.9mm_P5.00mm, F.Cu at (331.2, 130.0)
- added C31: 100n, Capacitor_THT:C_Disc_D4.3mm_W1.9mm_P5.00mm, F.Cu at (331.2, 149.3)
- added C4: 100n, Capacitor_THT:C_Disc_D4.3mm_W1.9mm_P5.00mm, F.Cu at (83.8, 72.0)
- added C5: 100n, Capacitor_THT:C_Disc_D4.3mm_W1.9mm_P5.00mm, F.Cu at (87.9, 110.7)
- added C6: 100n, Capacitor_THT:C_Disc_D4.3mm_W1.9mm_P5.00mm, F.Cu at (87.9, 129.8)
- added C7: 100n, Capacitor_THT:C_Disc_D4.3mm_W1.9mm_P5.00mm, F.Cu at (87.8, 148.8)
- added C8: 100n, Capacitor_THT:C_Disc_D4.3mm_W1.9mm_P5.00mm, F.Cu at (75.4, 173.1)
- added C9: 100n, Capacitor_THT:C_Disc_D4.3mm_W1.9mm_P5.00mm, F.Cu at (85.7, 204.2)
- added J11: Data bus, Connector_IDC:IDC-Header_2x08_P2.54mm_Vertical, F.Cu at (309.9, 157.0)
- added J12: A7 B1, Connector_PinHeader_2.54mm:PinHeader_1x02_P2.54mm_Vertical, F.Cu at (238.5, 53.7)
- added J2: Voltage test port, Connector_Wago:Wago_734-134_1x04_P3.50mm_Vertical, F.Cu at (40.1, 45.6)
- added J3: CLK, Connector_PinHeader_2.54mm:PinHeader_1x01_P2.54mm_Vertical, F.Cu at (275.3, 140.6)
- added J4: INR CPL, Connector_PinHeader_2.54mm:PinHeader_1x08_P2.54mm_Vertical, F.Cu at (372.0, 107.6)
- added J5: D5 E8, Connector_PinHeader_2.54mm:PinHeader_1x02_P2.54mm_Vertical, F.Cu at (275.3, 119.8)
- added J6: External control, Connector_PinSocket_2.54mm:PinSocket_1x05_P2.54mm_Vertical, F.Cu at (97.4, 185.0)
- added J7: Conn_01x03_Pin, Connector_PinHeader_2.54mm:PinHeader_1x03_P2.54mm_Vertical, F.Cu at (368.6, 158.1)
- added J8: J3 E6 D6 D7, Connector_PinHeader_2.54mm:PinHeader_1x04_P2.54mm_Vertical, F.Cu at (94.7, 136.9)
- added J9: Address bus, Connector_IDC:IDC-Header_2x20_P2.54mm_Vertical, F.Cu at (206.8, 119.9)
- added U_A3: 74LS244, Package_DIP:DIP-20_W7.62mm, F.Cu at (359.5, 84.7)
- added U_B4: 74LS244, Package_DIP:DIP-20_W7.62mm, F.Cu at (315.0, 104.6)
- J1: value B1 -> WR RD; footprint Connector_Wire:SolderWire-0.1sqmm_1x01_D0.4mm_OD1mm -> Connector_PinHeader_2.54mm:PinHeader_1x02_P2.54mm_Vertical
- moved R5 40.8 mm to (256.2, 99.2), turned to 0 degrees
- moved SW3 35.1 mm to (283.0, 145.8), turned to -90 degrees
- moved C2 30.1 mm to (324.9, 212.8), turned to 0 degrees
- moved C3 30.0 mm to (325.1, 32.7), turned to 0 degrees
- moved R3 26.6 mm to (47.2, 151.0), turned to 0 degrees
- moved R7 24.7 mm to (287.7, 88.1), turned to -90 degrees
- moved R6 20.6 mm to (284.1, 88.1), turned to -90 degrees
- moved R2 9.65 mm to (36.7, 111.6)
- moved R8 8.78 mm to (231.9, 56.4)
- moved D1 8.51 mm to (270.4, 125.5)
- moved C1 8.39 mm to (280.5, 133.1)
- moved SW2 3.60 mm to (34.0, 204.2)
- moved DIS1 3.53 mm to (34.0, 119.0)
- moved DIS2 3.53 mm to (34.0, 140.8)
- moved RN1 3.02 mm to (315.0, 120.3)
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Connections:
- net /NC_B1 renamed /Ext.RDIN
- net /~{RDRDY2} renamed /~{Sys.D_OUT}
- net Net-(U_E7-A->B) renamed /DIAGRD
- net Net-(U_J7-I0a) renamed /Ext.~{D_OUT}
- net Net-(U_J7-I0d) renamed /Ext.~{MEMSEL}
- net Net-(U_J8-I0b) renamed /Ext.DIAGRD
- P1 pad 34: -12V -> unconnected-(P1-Pin_34-Pad34)
- P1 pad 70: -12V -> unconnected-(P1-Pin_70-Pad70)
- SW2 pad 1: GND -> unconnected-(SW2-A-Pad1)
- SW3 pad 4: unconnected-(SW3-Pad4) -> Net-(J3-Pin_1)
- U_A4 pad 11: unconnected-(U_A4-I0b-Pad11) -> /HIGHMEM
- U_A4 pad 13: unconnected-(U_A4-I1b-Pad13) -> /PA16
- U_A4 pad 15: unconnected-(U_A4-I2b-Pad15) -> /PA17
- U_A4 pad 19: /LOW -> /HIGH
- U_A4 pad 5: unconnected-(U_A4-O2b-Pad5) -> /Sys.~{PA_{17}}
- U_A4 pad 7: unconnected-(U_A4-O1b-Pad7) -> /Sys.~{PA_{16}}
- U_A4 pad 9: unconnected-(U_A4-O0b-Pad9) -> /Sys.~{A_{15}}
- U_AB1 pad 13: unconnected-(U_AB1-Pad13) -> Net-(J1-Pin_2)
- U_B5 pad 1: Net-(U_B5-OE) -> /BUSRD
- U_B5 pad 11: /BUSRD -> /BUSWR_LE
- U_C4 pad 12: unconnected-(U_C4-Pad12) -> Net-(J5-Pin_1)
- U_C4 pad 13: unconnected-(U_C4-Pad13) -> Net-(J5-Pin_2)
- U_D1 pad 10: (no net) -> Net-(J12-Pin_2)
- U_D1 pad 11: (no net) -> /Sys.~{DRDY}
- U_D1 pad 8: (no net) -> Net-(J12-Pin_1)
- U_D1 pad 9: (no net) -> Net-(J12-Pin_2)
- U_J5 pad 10: unconnected-(U_J5-Pad10) -> Net-(J8-Pin_2)
- U_J5 pad 14: (no net) -> +5V
- U_J5 pad 6: unconnected-(U_J5-Pad6) -> Net-(J8-Pin_1)
- U_J5 pad 7: (no net) -> GND
- U_J6 pad 4: unconnected-(U_J6-Pad4) -> Net-(J8-Pin_4)
- U_J7 pad 11: unconnected-(U_J7-I0c-Pad11) -> /Ext.BUSRD
- U_J7 pad 7: /BUSRD -> /BUSWR_LE
- U_J7 pad 9: Net-(U_B5-OE) -> /BUSRD
- U_J8 pad 11: unconnected-(U_J8-I0c-Pad11) -> /Ext.~{MMIO}
- U_J8 pad 2: unconnected-(U_J8-I0a-Pad2) -> /Ext.~{DIAGWR}
Routing:
- net +5V: track 56.7 -> 1216.5 mm, vias 0 -> 1
- net GND: track 178.9 -> 939.7 mm, vias 0 -> 1
- net -12V: track 0.00 -> 395.6 mm, vias 0 -> 1
- net +12V: track 0.00 -> 381.9 mm, vias 0 -> 1
- net Net-(U_B5-OE): track 270.7 -> 0.00 mm, vias 1 -> 0
- net /BUSWR_LE: track 0.00 -> 230.0 mm, vias 0 -> 1
- net /HIGH: track 344.8 -> 545.2 mm, vias 2 -> 3
- net /A9: track 492.1 -> 577.4 mm, vias 1 -> 2
- net /Sys.~{DRDY}: track 88.0 -> 173.2 mm
- net /A0: track 590.8 -> 670.9 mm, vias 0 -> 1
- net /A10: track 449.8 -> 529.4 mm, vias 1 -> 2
- net /A8: track 496.9 -> 574.7 mm, vias 0 -> 3
- net /A1: track 570.6 -> 647.8 mm, vias 0 -> 1
- net /HIGHMEM: track 0.00 -> 75.4 mm
- net /A2: track 582.8 -> 657.0 mm, vias 1 -> 2
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Other:
- board text added: "+12V GND +5V -12V"

Commit message: DiagBoard, MUX: Verified space for puller tabs
Board layouts allow for two tabs, reserve space for both. Removed pre-defined
holes because tabs can be different depending on where they were ordered, it's
easier to drill two custom holes on the spot
Parts:
- removed REF** (x4): MountingHole_2.5mm, MountingHole:MountingHole_2.5mm
- moved SW2 25.6 mm to (34.0, 178.6)
- moved R2 24.0 mm to (36.8, 87.6)
- moved J2 18.9 mm to (40.3, 64.5)
- moved RN2 17.7 mm to (40.1, 149.3)
- moved SW1 17.7 mm to (25.9, 154.3)
- moved DIS1 17.7 mm to (34.0, 101.3)
- moved DIS2 17.7 mm to (34.0, 123.1)
- moved R3 17.7 mm to (47.2, 133.3)
- moved R4 4.17 mm to (59.1, 93.7)
- moved R8 0.89 mm to (231.9, 55.5)
Connections:
- SW2 pad 6: unconnected-(SW2-C-Pad6) -> GND
Routing:
- net Net-(U_J2-Q7): track 82.5 -> 61.2 mm
- net /D7_O: track 429.3 -> 448.9 mm, vias 2 -> 1
- net +12V: track 381.9 -> 400.9 mm
- net -12V: track 395.6 -> 414.5 mm
- net /D6_O: track 417.1 -> 435.2 mm
- net /D2_O: track 410.9 -> 428.9 mm
- net Net-(RN2-R5): track 21.6 -> 39.5 mm
- net /D3_O: track 400.7 -> 418.5 mm
- net /D5_O: track 434.2 -> 452.0 mm
- net /~{STRB}: track 166.0 -> 183.8 mm
- net Net-(U_J2-Q4): track 99.4 -> 81.7 mm
- net /D1_O: track 428.5 -> 446.3 mm
- net Net-(RN2-R2): track 24.2 -> 40.8 mm
- net /BLNK: track 134.7 -> 118.2 mm
- net Net-(RN2-R6): track 23.9 -> 40.1 mm
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
Commit message: DiagBoard: Add memory delay selection jumper
For experiments and fine-tuning.
Parts:
- added JP1: Memory delay select, Connector_PinHeader_2.54mm:PinHeader_2x08_P2.54mm_Vertical, F.Cu at (209.0, 60.5)
- moved R8 17.7 mm to (249.4, 58.0), turned to 0 degrees
- moved C18 1.17 mm to (230.1, 110.7)
Connections:
- U_E2 pad 10: unconnected-(U_E2-Qe-Pad10) -> Net-(JP1-A5)
- U_E2 pad 11: unconnected-(U_E2-Qf-Pad11) -> Net-(JP1-A6)
- U_E2 pad 12: unconnected-(U_E2-Qg-Pad12) -> Net-(JP1-A7)
- U_E2 pad 13: unconnected-(U_E2-Qh-Pad13) -> Net-(JP1-A8)
- U_E2 pad 4: unconnected-(U_E2-Qb-Pad4) -> Net-(JP1-A2)
- U_E2 pad 5: /DRDY -> Net-(JP1-A3)
- U_E2 pad 6: unconnected-(U_E2-Qd-Pad6) -> Net-(JP1-A4)
Routing:
- net +5V: track 1219.2 -> 1260.1 mm
- net Net-(JP1-A5): track 0.00 -> 17.7 mm
- net Net-(JP1-A7): track 0.00 -> 17.6 mm
- net Net-(JP1-A6): track 0.00 -> 17.3 mm
- net /DRDY: track 333.3 -> 316.4 mm
- net /HIGH: track 546.4 -> 529.9 mm
- net Net-(JP1-A2): track 0.00 -> 16.1 mm
- net /SR1: track 188.9 -> 204.9 mm
- net Net-(JP1-A8): track 0.00 -> 15.2 mm
- net Net-(JP1-A4): track 0.00 -> 12.9 mm
- net /RDWR: track 135.4 -> 146.5 mm
- net /~{MMIO}: track 95.6 -> 105.8 mm
- net GND: track 945.7 -> 953.2 mm
- net /A9: track 577.4 -> 583.5 mm
- net Net-(JP1-A3): track 0.00 -> 5.46 mm
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