File: DiagBoard/DiagBoard.kicad_pcb (KiCad board)
At the start: 4 copper layers, 364 x 203 mm, 104 parts, among them J1 WR RD, J11 Data bus, J12 A7 B1, J2 Voltage test port, J3 CLK, J4 INR CPL, J5 D5 E8, J6 External control, J7 Conn_01x03_Pin, J8 J3 E6 D6 D7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

Commit message: DiagBoard: Add /RESET to experimental connector
Can be useful
Parts:
- J7: footprint Connector_PinHeader_2.54mm:PinHeader_1x03_P2.54mm_Vertical -> Connector_PinHeader_2.54mm:PinHeader_1x04_P2.54mm_Vertical
- U_A2, U_A3, U_B4: value 74LS244 -> 74LS240
- moved J7 8.09 mm to (368.6, 166.2)
- moved R6 0.31 mm to (284.1, 87.8)
- moved R7 0.31 mm to (287.6, 87.8)
Connections:
- P1 pad 32: unconnected-(P1-Pin_32-Pad32) -> /~{Sys.Reset}
Routing:
- net +5V: track 1260.1 -> 1311.9 mm
- net GND: track 953.2 -> 984.3 mm
- net /D0_O: track 473.4 -> 489.3 mm, vias 1 -> 0
- net /~{Sys.Reset}: track 0.00 -> 13.8 mm
- net /Sys.~{APRE}: track 76.7 -> 68.4 mm
- net Net-(RN2-R3): track 40.8 -> 47.4 mm
- net /D3_O: track 418.5 -> 413.1 mm, vias 0 -> 1
- net Net-(D1-A): track 394.1 -> 388.8 mm
- net /Sys.~{D_{1}}: track 52.8 -> 47.7 mm
- net Net-(U_J2-Q4): track 81.7 -> 86.8 mm
- net /Sys.~{MEMFLT}: track 12.7 -> 17.7 mm
- net /Sys.~{INTRQ}: track 13.3 -> 18.1 mm
- net /Sys.~{RDIN}: track 163.9 -> 160.4 mm
- net /D5_O: track 452.0 -> 455.5 mm, vias 1 -> 0
- net /Sys.~{DRDY}: track 173.2 -> 169.9 mm
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