File: DiagBoard/DiagBoard.kicad_sch (KiCad schematic)
At the start: 104 parts, among them J1 WR RD, J11 Data bus, J12 A7 B1, J2 Voltage test port, J3 CLK, J4 INR CPL, J5 D5 E8, J6 External control, J7 Conn_01x03_Pin, J8 J3 E6 D6 D7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

Commit message: DiagBoard: Add /RESET to experimental connector
Can be useful
Parts:
- J7: footprint Connector_PinHeader_2.54mm:PinHeader_1x03_P2.54mm_Vertical -> Connector_PinHeader_2.54mm:PinHeader_1x04_P2.54mm_Vertical; symbol Connector:Conn_01x03_Pin -> Connector:Conn_01x04_Pin
- U_A2, U_A3, U_B4: value 74LS244 -> 74LS240
Connections:
- net ~{Sys.Reset}: now reaches P1.32 (Pin_32)
- net ~{Sys.Reset}: now also J7.4 (Pin_4)
- no-connect marks 59 -> 58
Changed lines of the file:
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@@
 	)
 	(no_connect
-		(at 711.2 322.58)
-	)
-	(no_connect
 		(at 626.11 222.25)
 	)
@@
 		)
 	)
+	(wire
+		(pts
+			(xy 701.04 337.82) (xy 765.81 337.82)
+		)
+		(stroke
+			(width 0)
+			(type default)
+		)
+	)
 	(bus
 		(pts
@@
 	(wire
 		(pts
+			(xy 765.81 337.82) (xy 765.81 317.5)
+		)
+		(stroke
+			(width 0)
+			(type default)
+		)
+	)
+	(wire
+		(pts
 			(xy 300.99 370.84) (xy 300.99 378.46)
 		)
@@
 	(wire
 		(pts
+			(xy 701.04 322.58) (xy 701.04 337.82)
+		)
+		(stroke
+			(width 0)
+			(type default)
+		)
+	)
+	(wire
+		(pts
 			(xy 519.43 322.58) (xy 497.84 322.58)
 		)
@@
 		)
 	)
+	(wire
+		(pts
+			(xy 701.04 322.58) (xy 711.2 322.58)
+		)
+		(stroke
+			(width 0)
+			(type default)
+		)
+	)
 	(bus
 		(pts
@@
 		)
 	)
+	(label "~{Sys.Reset}"
+		(at 701.04 337.82 0)
+		(effects
+			(font
+				(size 1.27 1.27)
+			)
+			(justify left bottom)
+		)
+	)
 	(label "A5"
 		(at 346.71 408.94 0)
@@
 			)
 		)
-		(property "Value" "74LS244"
+		(property "Value" "74LS240"
 			(at 642.2233 450.85 0)
 			(effects
@@
 			)
 		)
-		(property "Value" "74LS244"
+		(property "Value" "74LS240"
 			(at 641.9281 100.33 0)
 			(effects
@@
 	)
 	(symbol
-		(lib_id "Connector:Conn_01x03_Pin")
+		(lib_id "Connector:Conn_01x04_Pin")
 		(at 770.89 312.42 0)
 		(mirror y)
@@
 		(fields_autoplaced yes)
 		(property "Reference" "J7"
-			(at 772.16 311.1499 0)
+			(at 772.16 312.4199 0)
 			(effects
 				(font
@@
 		)
 		(property "Value" "Conn_01x03_Pin"
-			(at 772.16 313.6899 0)
+			(at 772.16 314.9599 0)
 			(effects
 				(font
@@
 			)
 		)
-		(property "Footprint" "Connector_PinHeader_2.54mm:PinHeader_1x03_P2.54mm_Vertical"
+		(property "Footprint" "Connector_PinHeader_2.54mm:PinHeader_1x04_P2.54mm_Vertical"
 			(at 770.89 312.42 0)
 			(effects
@@
 			)
 		)
-		(property "Description" "Generic connector, single row, 01x03, script generated"
+		(property "Description" "Generic connector, single row, 01x04, script generated"
 			(at 770.89 312.42 0)
 			(effects
@@
 		(pin "1"
 		)
+		(pin "4"
+		)
 		(instances
 			(project ""
@@
 			)
 		)
-		(property "Value" "74LS244"
+		(property "Value" "74LS240"
 			(at 640.9533 154.94 0)
 			(effects
