File: CPU/CPU.kicad_sch (KiCad schematic)
At the start: 211 parts, among them J1 Conn_02x36_Top_Bottom, P2 Conn_02x13_Top_Bottom, P3 Conn_02x13_Top_Bottom, P4 IDC-16, P5 Conn_02x25_Counter_Clockwise, P6 Conn_02x25_Counter_Clockwise, P7 Conn_02x07_Counter_Clockwise, P8 Conn_02x08_Odd_Even

Commit message: CPU: Support 28C16 ROMs
Add support for reconfiguring connections to support 28C16 ROM chips.
Parts:
- added JP2: ROM type select, Connector_PinHeader_2.54mm:PinHeader_1x03_P2.54mm_Vertical, symbol Jumper:Jumper_3_Bridged12
- added JP3: Conn_01x01_Female, Connector_Wire:SolderWire-0.1sqmm_1x01_D0.4mm_OD1mm, symbol Connector:Conn_01x01_Female
- added R26: 1K, Resistor_THT:R_Axial_DIN0207_L6.3mm_D2.5mm_P10.16mm_Horizontal, symbol Device:R
Connections:
- net +5V: now also R26.1
- net GND: now also JP3.1 (Pin_1)
- net MWS.A_{10}: now also JP2.2 (C); no longer U_MWE2.21 (A10), U_MWF2.21 (A10), U_MWH2.21 (A10), U_MWJ2.21 (A10), U_MWK2.21 (A10), U_MWL2.21 (A10), U_MWM2.21 (A10)
- net ~{ClockB_{0}}: now also P8.6 (Pin_6)
- net at R11.2, U_MWE2.18 (CE_{3}), U_MWF2.18 (CE_{3})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: no longer P8.6 (Pin_6)
- net at R10.2, U_MWE2.19 (CE_{2}), U_MWF2.19 (CE_{2})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: now also JP2.3 (B)
- new net: JP2.1 (A), R26.2, U_MWE2.21 (A10), U_MWF2.21 (A10), U_MWH2.21 (A10), U_MWJ2.21 (A10), U_MWK2.21 (A10), U_MWL2.21 (A10), U_MWM2.21 (A10)
Other:
- note added: "76161 ROMs: Install R10, R11; JP2 as shown; do not place R26 28C16 ROMs: Install R26; JP2 in opposite position; do not place R10, R11; connect pin 18 to ground using JP3"
- moved on the sheet: R10, R11

Commit message: CPU: Erratum E003
Found and fixed a missing connection
Connections:
- net Address.A_{8}: now also U_A6.11 (I0b)
- no-connect marks 93 -> 94
Changed lines of the file:
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@@
   (no_connect (at 695.96 335.28))
   (no_connect (at 45.72 459.74))
+  (no_connect (at 111.76 410.21))
   (no_connect (at 1112.52 166.37))
   (no_connect (at 318.77 311.15))
@@
     (stroke (width 0) (type default) (color 0 0 0 0))
   )
-  (wire (pts (xy 474.98 750.57) (xy 474.98 751.84))
-    (stroke (width 0) (type default) (color 0 0 0 0))
-  )
   (wire (pts (xy 212.09 143.51) (xy 213.36 143.51))
     (stroke (width 0) (type default) (color 0 0 0 0))
@@
     (effects (font (size 1.27 1.27)) (justify left bottom))
   )
+  (label "Address.A_{8}" (at 154.94 501.65 0)
+    (effects (font (size 1.27 1.27)) (justify left bottom))
+  )

Commit message: CPU: Synchronize footprints
Update footprint info from the PCB
Parts:
- C18, C31: footprint Capacitor_THT:C_Rect_L9.0mm_W2.5mm_P7.50mm_MKT -> Capacitor_THT:C_Disc_D4.3mm_W1.9mm_P5.00mm
Changed lines of the file:
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@@
       (effects (font (size 1.27 1.27)) (justify left))
     )
-    (property "Footprint" "Capacitor_THT:C_Rect_L9.0mm_W2.5mm_P7.50mm_MKT" (id 2) (at 1060.45 660.4 0)
+    (property "Footprint" "Capacitor_THT:C_Disc_D4.3mm_W1.9mm_P5.00mm" (id 2) (at 1060.45 660.4 0)
       (effects (font (size 1.27 1.27)) hide)
     )
@@
       (effects (font (size 1.27 1.27)) (justify left))
     )
-    (property "Footprint" "Capacitor_THT:C_Rect_L9.0mm_W2.5mm_P7.50mm_MKT" (id 2) (at 1066.8 683.26 0)
+    (property "Footprint" "Capacitor_THT:C_Disc_D4.3mm_W1.9mm_P5.00mm" (id 2) (at 1066.8 683.26 0)
       (effects (font (size 1.27 1.27)) hide)
     )
@@
     )
     (path "/077e4de8-86f6-4f35-aee2-3bd824b045da"
-      (reference "C18") (unit 1) (value "100nF") (footprint "Capacitor_THT:C_Rect_L9.0mm_W2.5mm_P7.50mm_MKT")
+      (reference "C18") (unit 1) (value "100nF") (footprint "Capacitor_THT:C_Disc_D4.3mm_W1.9mm_P5.00mm")
     )
     (path "/55e75c13-072a-4aec-9bc6-b21da459b850"
@@
     )
     (path "/094e65e7-3049-42a8-9da8-2d2f6d3b87e5"
-      (reference "C31") (unit 1) (value "100nF") (footprint "Capacitor_THT:C_Rect_L9.0mm_W2.5mm_P7.50mm_MKT")
+      (reference "C31") (unit 1) (value "100nF") (footprint "Capacitor_THT:C_Disc_D4.3mm_W1.9mm_P5.00mm")
     )
     (path "/a5cde810-ca8f-4d48-ac8a-3bea64b8b1d2"

Commit message: CPU: Microcode ROM override signal
P7 pin 14, the same as in original. Extremely useful for testing. Since 28c16
uses zero-active CE, make use of a spare inverter.
Parts:
- removed JP3: Conn_01x01_Female, Connector_Wire:SolderWire-0.1sqmm_1x01_D0.4mm_OD1mm, symbol Connector:Conn_01x01_Female
- removed R11: 1k, Resistor_THT:R_Axial_DIN0207_L6.3mm_D2.5mm_P10.16mm_Horizontal, symbol Device:R
- added JP3: ROM type select, Connector_PinHeader_2.54mm:PinHeader_1x03_P2.54mm_Vertical, symbol Jumper:Jumper_3_Bridged12
- added R4: 1k, Resistor_THT:R_Axial_DIN0207_L6.3mm_D2.5mm_P10.16mm_Horizontal, symbol Device:R
- R26: now not fitted
Connections:
- net +5V: now also R4.1
- net GND: no longer U_L14.1, U_L14.2
- net ~{MWROMEN}: now reaches U_L14.3
- net ~{MWROMEN}: now also JP3.3 (B)
- net at U_MWE2.18 (CE_{3}), U_MWF2.18 (CE_{3}), U_MWH2.18 (CE_{3})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: now also JP3.2 (C)
- net MWROMEN: now reaches P7.14 (Pin_14)
- net MWROMEN: now also U_L14.1, U_L14.2, JP3.1 (A), R4.2
- no-connect marks 94 -> 92
Other:
- note added: "76161 ROMs: Install R10; JP2 and JP3 as shown; do not place R26 28C16 ROMs: Install R26; JP2 and JP3 in opposite position; do not place R10"
- note removed: "76161 ROMs: Install R10, R11; JP2 as shown; do not place R26 28C16 ROMs: Install R26; JP2 in opposite position; do not place R10, R11; connect pin 18 to ground using JP3"
- moved on the sheet: R10, U_L14A
